File: hardware/gateway/gateway.kicad_pcb (KiCad board)
At the start: 2 copper layers, 0 parts

Commit message: EG-12 Components placed without connections. Balun components place needs to be fixed.
Parts:
- added ANT1: ANT-868-HESM, MyParts:ANT-868-HESM, F.Cu at (187.7, 142.5)
- added C1: 100nF, Capacitor_SMD:C_0603_1608Metric, F.Cu at (143.9, 153.8)
- added C10: 1uF, Capacitor_SMD:C_0603_1608Metric, F.Cu at (155.6, 126.2)
- added C11: 100nF, Capacitor_SMD:C_0603_1608Metric, F.Cu at (152.3, 126.2)
- added C12: 100nF, Capacitor_SMD:C_0603_1608Metric, F.Cu at (149.7, 131.7)
- added C121: 1pF, Capacitor_SMD:C_0402_1005Metric, F.Cu at (161.9, 131.2)
- added C122: 1.5pF, Capacitor_SMD:C_0402_1005Metric, F.Cu at (166.1, 129.2)
- added C123: 3.3pF, Capacitor_SMD:C_0402_1005Metric, F.Cu at (170.8, 128.0)
- added C124: 100pF, Capacitor_SMD:C_0402_1005Metric, F.Cu at (162.8, 126.3)
- added C125: 12pF, Capacitor_SMD:C_0402_1005Metric, F.Cu at (174.6, 130.6)
- added C13: 12pF, Capacitor_SMD:C_0402_1005Metric, F.Cu at (150.3, 136.0)
- added C131: 1.5pF, Capacitor_SMD:C_0402_1005Metric, F.Cu at (162.6, 133.5)
- added C14: 12pF, Capacitor_SMD:C_0402_1005Metric, F.Cu at (157.6, 136.1)
- added C15: 22uF, 6.3V, Capacitor_SMD:C_1206_3216Metric, F.Cu at (108.4, 156.3)
- added C16: 4.7pF, Capacitor_SMD:C_0402_1005Metric, F.Cu at (127.3, 153.8)
- added C17: 4.7uF, 25V, Capacitor_SMD:C_0805_2012Metric, F.Cu at (137.5, 156.8)
- added C18: 4.7uF, 25V, Capacitor_SMD:C_0805_2012Metric, F.Cu at (104.4, 136.8)
- added C19: 100nF, Capacitor_SMD:C_0603_1608Metric, F.Cu at (104.6, 147.8)
- added C2: 100nF, Capacitor_SMD:C_0603_1608Metric, F.Cu at (105.3, 127.9)
- added C3: 10nF, Capacitor_SMD:C_0402_1005Metric, F.Cu at (85.0, 130.7)
- added C4: 1uF, Capacitor_SMD:C_0603_1608Metric, F.Cu at (86.2, 141.5)
- added C5: 100nF, Capacitor_SMD:C_0603_1608Metric, F.Cu at (90.8, 141.5)
- added C6: 47uF, 6.3V, Capacitor_SMD:C_1206_3216Metric, F.Cu at (83.3, 137.7)
- added C7: 1uF, Capacitor_SMD:C_0603_1608Metric, F.Cu at (93.6, 150.8)
- added C8: 100nF, Capacitor_SMD:C_0603_1608Metric, F.Cu at (96.0, 150.9)
- added C9: 47uF, 6.3V, Capacitor_SMD:C_1206_3216Metric, F.Cu at (144.1, 134.4)
- added Csh1: 0, Capacitor_SMD:C_0603_1608Metric, F.Cu at (181.4, 136.2)
- added Csh2: 0, Capacitor_SMD:C_0603_1608Metric, F.Cu at (176.3, 136.3)
- added D1: MBR0520LT3G, MyParts:SOD3716X135N, F.Cu at (119.9, 156.2)
- added FB1: BLM18KG601SN1D, MyParts:BLM18SP221SN1B, F.Cu at (143.3, 130.0)
- added IC1: STM8L151K4T6, MyParts:QFP80P900X900X160-32N, F.Cu at (94.4, 133.0)
- added IC2: CC1101RGPR, MyParts:QFN50P400X400X100-21N-D, F.Cu at (154.0, 130.7)
- added IC3: LT1615ES5-1#TRMPBF, MyParts:SOT95P280X100-5N, F.Cu at (127.8, 157.1)
- added IC4: MIC4427YM, MyParts:SOIC127P599X173-8N, F.Cu at (105.4, 142.5)
- added IC5: MB85RC64TAPNF-G-BDERE1, MyParts:SOIC127P602X173-8N, F.Cu at (87.7, 152.0)
- added J1: G8250041000YEU, MyParts:HDRV4W55P0X200_1X4_800X200X635P, F.Cu at (142.3, 126.5)
- added J2: M20-9770342, MyParts:HDRV3W66P0X254_1X3_762X254X855P, F.Cu at (153.4, 152.7)
- added L121: 12nH, Inductor_SMD:L_0402_1005Metric, F.Cu at (159.8, 129.3)
- added L122: 18nH, Inductor_SMD:L_0402_1005Metric, F.Cu at (162.7, 128.7)
- added L123: 12nH, Inductor_SMD:L_0402_1005Metric, F.Cu at (169.4, 130.6)
- added L124: 12nH, Inductor_SMD:L_0402_1005Metric, F.Cu at (171.9, 130.6)
- added L131: 12nH, Inductor_SMD:L_0402_1005Metric, F.Cu at (159.6, 133.1)
- added L132: 18nH, Inductor_SMD:L_0402_1005Metric, F.Cu at (166.2, 132.0)
- added L2: CD43NP-100MC, MyParts:CD43NP100MC, F.Cu at (114.5, 156.6)
- added LED1: WP710A10LVBC_D, MyParts:WP710A10LVBCD, F.Cu at (162.7, 143.3)
- added LED2: TLHY4400-AS12Z, MyParts:TLHY4400AS12Z, F.Cu at (157.4, 143.3)
- added LED3: TLHR4400-AS12Z, MyParts:TLHR4400AS12Z, F.Cu at (151.9, 143.5)
- added LS1: PKMCS1818E20A0-R1, MyParts:PKMCS1818E20A0R1, F.Cu at (125.5, 142.7)
- added Q1: IRLML6402TRPBF, MyParts:SOT95P237X112-3N, F.Cu at (128.8, 129.1)
- added R1: 100K, Resistor_SMD:R_0402_1005Metric, F.Cu at (133.3, 129.0)
- added R10: 50, Resistor_SMD:R_0402_1005Metric, F.Cu at (152.0, 146.9)
- added R11: 10K, Resistor_SMD:R_0402_1005Metric, F.Cu at (96.3, 154.3)
- added R12: 10K, Resistor_SMD:R_0402_1005Metric, F.Cu at (93.5, 155.9)
- added R13: 56K, Resistor_SMD:R_0402_1005Metric, F.Cu at (158.1, 126.5)
- added R14: 0R, Resistor_SMD:R_0603_1608Metric, F.Cu at (179.0, 135.5)
- added R15: 100K, Resistor_SMD:R_0402_1005Metric, F.Cu at (124.8, 156.6)
- added R16: 130K, Resistor_SMD:R_0402_1005Metric, F.Cu at (131.8, 158.4)
- added R17: 1.15M, Resistor_SMD:R_0402_1005Metric, F.Cu at (132.8, 155.1)
- added R18: 33R, Resistor_SMD:R_0402_1005Metric, F.Cu at (112.1, 140.5)
- added R19: 33R, Resistor_SMD:R_0402_1005Metric, F.Cu at (112.0, 144.4)
- added R2: 1M, Resistor_SMD:R_0402_1005Metric, F.Cu at (146.6, 155.0)
- added R20: 1M, Resistor_SMD:R_0402_1005Metric, F.Cu at (114.0, 142.7)
- added R3: 100K, Resistor_SMD:R_0402_1005Metric, F.Cu at (146.7, 153.1)
- added R4: 10K, Resistor_SMD:R_0402_1005Metric, F.Cu at (145.2, 150.1)
- added R5: 1M, Resistor_SMD:R_0402_1005Metric, F.Cu at (110.5, 128.1)
- added R6: 510K, Resistor_SMD:R_0402_1005Metric, F.Cu at (115.2, 128.2)
- added R7: 1K, Resistor_SMD:R_0402_1005Metric, F.Cu at (119.8, 128.3)
- added R8: 100, Resistor_SMD:R_0402_1005Metric, F.Cu at (162.6, 146.3)
- added R9: 50, Resistor_SMD:R_0402_1005Metric, F.Cu at (157.5, 147.5)
- added S1: MASM-14R-8-10, MyParts:MASM14R810, F.Cu at (152.9, 158.1)
- added S2: B3F-1070, MyParts:B3F1060, F.Cu at (144.8, 143.1)
- added U1: 2462, MyParts:2462, B.Cu at (137.1, 135.2)
- added Y1: NX3225GA-26.000M-STD-CRG-2, MyParts:NX3225GA26000MSTDCRG2, F.Cu at (154.0, 135.9)
Routing:
- net Net-(IC2-XOSC_Q1): track 0.00 -> 7.89 mm
- net Net-(IC2-XOSC_Q2): track 0.00 -> 2.64 mm
- net GND: track 0.00 -> 2.58 mm
Other:
- board outline added: 124 x 36 mm
