File: hardware/gateway/buzzer.kicad_sch (KiCad schematic)
At the start: 16 parts, among them IC3 LT1615ES5-1#TRMPBF, IC4 MIC4427YM

Commit message: EG-11 All components connected in all sheets. The MCU pin mapping needs to be fixed. The BOM needs to be created. The FRAM need needs to be assessed.
Parts:
- C1: value 10uF, 6.3V -> 22uF, 6.3V
Changed lines of the file:
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@@
 			)
 		)
-		(property "Value" "10uF, 6.3V"
+		(property "Value" "22uF, 6.3V"
 			(at 46.99 50.7999 0)
 			(effects

Commit message: EG-11 BOM generated.
Parts:
- removed C1: 22uF, 6.3V, symbol Device:C
- removed C2, C8: 4.7uF, 25V, symbol Device:C
- removed C3: 4.7pF, symbol Device:C
- removed C9: 100nF, symbol Device:C
- removed R12: 100K, symbol Device:R_US
- removed R21: 33, symbol Device:R_US
- added C15: 22uF, 6.3V, Capacitor_SMD:C_1206_3216Metric, symbol Device:C
- added C16: 4.7pF, Capacitor_SMD:C_0402_1005Metric, symbol Device:C
- added C17, C18: 4.7uF, 25V, Capacitor_SMD:C_0805_2012Metric, symbol Device:C
- added C19: 100nF, Capacitor_SMD:C_0603_1608Metric, symbol Device:C
- added R15: 100K, Resistor_SMD:R_0402_1005Metric, symbol Device:R_US
- added R16: 130K, Resistor_SMD:R_0402_1005Metric, symbol Device:R_US
- R17: footprint (none) -> Resistor_SMD:R_0402_1005Metric; Manufacturer_Name (none) -> Yageo; Manufacturer_Part_Number (none) -> RC0402FR-071M15L; Mouser Part Number (none) -> 603-RC0402FR-071M15L; Mouser Price/Stock (none) -> https://pt.mouser.com/ProductDetail/YAGEO/RC0402FR-071M15L?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
- R18: value 130K -> 33R; footprint (none) -> Resistor_SMD:R_0402_1005Metric; Manufacturer_Name (none) -> Panasonic; Manufacturer_Part_Number (none) -> ERJ-S02J330X; Mouser Part Number (none) -> 667-ERJ-S02J330X; Mouser Price/Stock (none) -> https://pt.mouser.com/ProductDetail/Panasonic/ERJ-S02J330X?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
- R19: value 1M -> 33R; footprint (none) -> Resistor_SMD:R_0402_1005Metric; Manufacturer_Name (none) -> Panasonic; Manufacturer_Part_Number (none) -> ERJ-S02J330X; Mouser Part Number (none) -> 667-ERJ-S02J330X; Mouser Price/Stock (none) -> https://pt.mouser.com/ProductDetail/Panasonic/ERJ-S02J330X?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
- R20: value 33 -> 1M; footprint (none) -> Resistor_SMD:R_0402_1005Metric; Manufacturer_Name (none) -> Yageo; Manufacturer_Part_Number (none) -> RC0402JR-7D1ML; Mouser Part Number (none) -> 603-RC0402JR-7D1ML; Mouser Price/Stock (none) -> https://pt.mouser.com/ProductDetail/YAGEO/RC0402JR-7D1ML?qs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
Connections:
- net +12V: now also C16.1, C17.1, C18.1, C19.1
- net BZR_EN: now also R15.2
- net GND: now also C15.2, C17.2, C18.2, C19.2, R15.1, R16.1; no longer R18.2
- net VDD: now also C15.1
- net at IC4.5 (OUTB): now also R19.2
- net at LS1.3 (-_1), LS1.4 (-_2): now also R19.1, R20.1; no longer R19.2
- net at IC3.3 (FB), R17.1: now also C16.2, R16.2; no longer R18.1
- net at LS1.1 (+_1), LS1.2 (+_2), R20.2: now also R18.1; no longer R19.1
- net at IC4.7 (OUTA): now also R18.2; no longer R20.1

Commit message: EG-11 ERC passed.
Changed lines of the file:
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@@
+	)
+	(junction
+		(at 129.54 38.1)
+		(diameter 0)
+		(color 0 0 0 0)
 	)
 	(junction
@@
 	(wire
 		(pts
+			(xy 135.89 38.1) (xy 129.54 38.1)
+		)
+		(stroke
+			(width 0)
+			(type default)
+		)
+	)
+	(wire
+		(pts
 			(xy 99.06 38.1) (xy 104.14 38.1)
 		)
@@
 		(pts
 			(xy 111.76 33.02) (xy 115.57 33.02)
+		)
+		(stroke
+			(width 0)
+			(type default)
+		)
+	)
+	(wire
+		(pts
+			(xy 135.89 36.83) (xy 135.89 38.1)
 		)
 		(stroke
@@
 					(unit 1)
 				)
+			)
+		)
+	)
+	(symbol
+		(lib_id "power:PWR_FLAG")
+		(at 135.89 36.83 0)
+		(unit 1)
+		(exclude_from_sim no)
+		(in_bom yes)
+		(on_board yes)
+		(dnp no)
+		(fields_autoplaced yes)
+		(property "Reference" "#FLG05"
+			(at 135.89 34.925 0)
+			(effects
+				(font
+					(size 1.27 1.27)
+				)
+				(hide yes)
+			)
+		)
+		(property "Value" "PWR_FLAG"
+			(at 135.89 31.75 0)
+			(effects
+				(font
+					(size 1.27 1.27)
+				)
+			)
+		)
+		(property "Footprint" ""
+			(at 135.89 36.83 0)
+			(effects
+				(font
+					(size 1.27 1.27)
+				)
+				(hide yes)
+			)
+		)
+		(property "Datasheet" "~"
+			(at 135.89 36.83 0)
+			(effects
+				(font
+					(size 1.27 1.27)
+				)
+				(hide yes)
+			)
+		)
+		(property "Description" "Special symbol for telling ERC where power comes from"
+			(at 135.89 36.83 0)
+			(effects
+				(font
+					(size 1.27 1.27)
+				)
+				(hide yes)
+			)
+		)
+		(pin "1"
+		)
+		(instances
+			(project ""
+				(path "/d3cb7130-decc-418b-958e-e5d84a8d867f/fe77db69-068b-4697-8152-e8993e362189"
+					(reference "#FLG05")
+					(unit 1)
+				)

Commit message: EG-12 All components placed. RF connected, except antenna. Buzzer connected, buzzer power supply connected, FRAM connected. Majority os MCU connections  missing.
Parts:
- removed C19: 100nF, Capacitor_SMD:C_0603_1608Metric, symbol Device:C
- added C24: 100nF, Capacitor_SMD:C_0402_1005Metric, symbol Device:C
- renumbered C15 to C20, C16 to C21, C17 to C22, C18 to C23
Connections:
- net +12V: now also C24.1
- net GND: now also C24.2
Changed lines of the file:
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@@
 		(on_board yes)
 		(dnp no)
-		(property "Reference" "C18"
+		(property "Reference" "C23"
 			(at 74.93 106.6799 0)
 			(effects
@@
 			(project "gateway"
 				(path "/d3cb7130-decc-418b-958e-e5d84a8d867f/fe77db69-068b-4697-8152-e8993e362189"
-					(reference "C18")
+					(reference "C23")
 					(unit 1)
 				)
@@
 		(dnp no)
 		(fields_autoplaced yes)
-		(property "Reference" "C17"
+		(property "Reference" "C22"
 			(at 119.38 45.7199 0)
 			(effects
@@
 			(project "gateway"
 				(path "/d3cb7130-decc-418b-958e-e5d84a8d867f/fe77db69-068b-4697-8152-e8993e362189"
-					(reference "C17")
+					(reference "C22")
 					(unit 1)
 				)
@@
 		(dnp no)
 		(fields_autoplaced yes)
-		(property "Reference" "C15"
+		(property "Reference" "C20"
 			(at 46.99 48.2599 0)
 			(effects
@@
 			(project "gateway"
 				(path "/d3cb7130-decc-418b-958e-e5d84a8d867f/fe77db69-068b-4697-8152-e8993e362189"
-					(reference "C15")
+					(reference "C20")
 					(unit 1)
 				)
@@
 	)
 	(symbol
+		(lib_id "Device:C")
+		(at 86.36 107.95 0)
+		(unit 1)
+		(exclude_from_sim no)
+		(in_bom yes)
+		(on_board yes)
+		(dnp no)
+		(fields_autoplaced yes)
+		(property "Reference" "C24"
+			(at 90.17 106.6799 0)
+			(effects
+				(font
+					(size 1.27 1.27)
+				)
+				(justify left)
+			)
+		)
+		(property "Value" "100nF"
+			(at 90.17 109.2199 0)
+			(effects
+				(font
+					(size 1.27 1.27)
+				)
+				(justify left)
+			)
+		)
+		(property "Footprint" "Capacitor_SMD:C_0402_1005Metric"
+			(at 87.3252 111.76 0)
+			(effects
+				(font
+					(size 1.27 1.27)
+				)
+				(hide yes)
+			)
+		)
+		(property "Datasheet" "~"
+			(at 86.36 107.95 0)
+			(effects
+				(font
+					(size 1.27 1.27)
+				)
+				(hide yes)
+			)
+		)
+		(property "Description" "Unpolarized capacitor"
+			(at 86.36 107.95 0)
+			(effects
+				(font
+					(size 1.27 1.27)
+				)
+				(hide yes)
+			)
+		)
+		(property "Mouser Part Number" "603-CC402KRX7R7BB104"
+			(at 86.36 107.95 0)
+			(effects
+				(font
+					(size 1.27 1.27)
+				)
+				(hide yes)
+			)
+		)
+		(property "Mouser Price/Stock" "https://pt.mouser.com/ProductDetail/YAGEO/CC0402KRX7R7BB104?qs=AgBp2OyFlx%252BSOyhfyS7hpw%3D%3D"
+			(at 86.36 107.95 0)
+			(effects
+				(font
+					(size 1.27 1.27)
+				)
+				(hide yes)
+			)
+		)
+		(property "Manufacturer_Name" "Yageo"
+			(at 86.36 107.95 0)
+			(effects
+				(font
+					(size 1.27 1.27)
+				)
+				(hide yes)
+			)
+		)
+		(property "Manufacturer_Part_Number" "CC0402KRX7R7BB104"
+			(at 86.36 107.95 0)
+			(effects
+				(font
+					(size 1.27 1.27)
+				)
+				(hide yes)
+			)
+		)
+		(pin "2"
+		)
+		(pin "1"
+		)
+		(instances
+			(project "gateway"
+				(path "/d3cb7130-decc-418b-958e-e5d84a8d867f/fe77db69-068b-4697-8152-e8993e362189"
+					(reference "C24")
+					(unit 1)
+				)
+			)
+		)
+	)
+	(symbol
 		(lib_id "power:GND")
 		(at 115.57 55.88 0)
@@
 				(path "/d3cb7130-decc-418b-958e-e5d84a8d867f/fe77db69-068b-4697-8152-e8993e362189"
 					(reference "#PWR027")
-					(unit 1)
-				)
-			)
-		)
-	)
-	(symbol
-		(lib_id "Device:C")
-		(at 86.36 107.95 0)
-		(unit 1)
-		(exclude_from_sim no)
-		(in_bom yes)
-		(on_board yes)
-		(dnp no)
-		(fields_autoplaced yes)
-		(property "Reference" "C19"
-			(at 90.17 106.6799 0)
-			(effects
-				(font
-					(size 1.27 1.27)
-				)
-				(justify left)
-			)
-		)
-		(property "Value" "100nF"
-			(at 90.17 109.2199 0)
-			(effects
-				(font
-					(size 1.27 1.27)
-				)
-				(justify left)
-			)
-		)
-		(property "Footprint" "Capacitor_SMD:C_0603_1608Metric"
-			(at 87.3252 111.76 0)
-			(effects
-				(font
-					(size 1.27 1.27)
-				)
-				(hide yes)
-			)
-		)
-		(property "Datasheet" "~"
-			(at 86.36 107.95 0)
-			(effects
-				(font
-					(size 1.27 1.27)
-				)
-				(hide yes)
-			)
-		)
-		(property "Description" "Unpolarized capacitor"
-			(at 86.36 107.95 0)
-			(effects
-				(font
-					(size 1.27 1.27)
-				)
-				(hide yes)
-			)
-		)
-		(property "Mouser Part Number" "81-GCJ188R72A104KA1D"
-			(at 86.36 107.95 0)
-			(effects
-				(font
-					(size 1.27 1.27)
-				)
-				(hide yes)
-			)
-		)
-		(property "Mouser Price/Stock" "https://pt.mouser.com/ProductDetail/Murata-Electronics/GCJ188R72A104KA01D?qs=vAU15TnRQM%2FvAWQMlXkQEQ%3D%3D"
-			(at 86.36 107.95 0)
-			(effects
-				(font
-					(size 1.27 1.27)
-				)
-				(hide yes)
-			)
-		)
-		(property "Manufacturer_Name" "Murata"
-			(at 86.36 107.95 0)
-			(effects
-				(font
-					(size 1.27 1.27)
-				)
-				(hide yes)
-			)
-		)
-		(property "Manufacturer_Part_Number" "GCJ188R72A104KA1D"
-			(at 86.36 107.95 0)
-			(effects
-				(font
-					(size 1.27 1.27)
-				)
-				(hide yes)
-			)
-		)
-		(pin "2"
-		)
-		(pin "1"
-		)
-		(instances
-			(project "gateway"
-				(path "/d3cb7130-decc-418b-958e-e5d84a8d867f/fe77db69-068b-4697-8152-e8993e362189"
-					(reference "C19")
 					(unit 1)
 				)
@@
 		(on_board yes)
 		(dnp no)
-		(property "Reference" "C16"
+		(property "Reference" "C21"
 			(at 106.68 26.67 90)
 			(effects
@@
 			(project "gateway"
 				(path "/d3cb7130-decc-418b-958e-e5d84a8d867f/fe77db69-068b-4697-8152-e8993e362189"
-					(reference "C16")
-					(unit 1)
-				)
+					(reference "C21")
+					(unit 1)
+				)

Commit message: EG-38 Replaced all BOM field names to proper ones, according with manufacturer standards.
Parts:
- C20: Manufacturer (none) -> Murata; Manufacturer Part Number (none) -> GGM31CD70J226KE02L; Manufacturer_Name Murata -> (none); Manufacturer_Part_Number GGM31CD70J226KE02L -> (none); Mouser Price/Stock https://pt.mouser.com/ProductDetail/Murata-Electronics/GGM3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 -> (none); Supplier Link (none) -> https://pt.mouser.com/ProductDetail/Murata-Electronics/GGM3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
- C21: Manufacturer (none) -> Murata; Manufacturer Part Number (none) -> GCM1555C2A4R7BE02D; Manufacturer_Name Murata -> (none); Manufacturer_Part_Number GCM1555C2A4R7BE02D -> (none); Mouser Price/Stock https://pt.mouser.com/ProductDetail/Murata-Electronics/GCM1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 -> (none); Supplier Link (none) -> https://pt.mouser.com/ProductDetail/Murata-Electronics/GCM1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
- C22, C23: Manufacturer (none) -> Taiyo Yuden; Manufacturer Part Number (none) -> MCAST21GBC7475KTCA01; Manufacturer_Name Taiyo Yuden -> (none); Manufacturer_Part_Number MCAST21GBC7475KTCA01 -> (none); Mouser Price/Stock https://pt.mouser.com/ProductDetail/TAIYO-YUDEN/MCAST21GBC7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 -> (none); Supplier Link (none) -> https://pt.mouser.com/ProductDetail/TAIYO-YUDEN/MCAST21GBC7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
- C24: Manufacturer (none) -> Yageo; Manufacturer Part Number (none) -> CC0402KRX7R7BB104; Manufacturer_Name Yageo -> (none); Manufacturer_Part_Number CC0402KRX7R7BB104 -> (none); Mouser Price/Stock https://pt.mouser.com/ProductDetail/YAGEO/CC0402KRX7R7BB104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 -> (none); Supplier Link (none) -> https://pt.mouser.com/ProductDetail/YAGEO/CC0402KRX7R7BB104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
- D1: Manufacturer (none) -> onsemi; Manufacturer Part Number (none) -> MBR0520LT3G; Manufacturer_Name onsemi -> (none); Manufacturer_Part_Number MBR0520LT3G -> (none); Mouser Price/Stock https://www.mouser.co.uk/ProductDetail/onsemi/MBR0520LT3G?q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 -> (none); Supplier Link (none) -> https://www.mouser.co.uk/ProductDetail/onsemi/MBR0520LT3G?q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
- IC3: Manufacturer (none) -> Analog Devices; Manufacturer Part Number (none) -> LT1615ES5-1#TRMPBF; Manufacturer_Name Analog Devices -> (none); Manufacturer_Part_Number LT1615ES5-1#TRMPBF -> (none); Mouser Price/Stock https://www.mouser.co.uk/ProductDetail/Analog-Devices/LT161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 -> (none); Supplier Link (none) -> https://www.mouser.co.uk/ProductDetail/Analog-Devices/LT161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
- IC4: Manufacturer (none) -> Microchip; Manufacturer Part Number (none) -> MIC4427YM; Manufacturer_Name Microchip -> (none); Manufacturer_Part_Number MIC4427YM -> (none); Mouser Price/Stock https://www.mouser.co.uk/ProductDetail/Microchip-Technology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 -> (none); Supplier Link (none) -> https://www.mouser.co.uk/ProductDetail/Microchip-Technology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
- L2: Manufacturer (none) -> Sumida; Manufacturer Part Number (none) -> CD43NP-100MC; Manufacturer_Name Sumida -> (none); Manufacturer_Part_Number CD43NP-100MC -> (none); Mouser Price/Stock https://www.mouser.co.uk/ProductDetail/Sumida/CD43NP-100MC?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 -> (none); Supplier Link (none) -> https://www.mouser.co.uk/ProductDetail/Sumida/CD43NP-100MC?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
- LS1: Manufacturer (none) -> Murata Electronics; Manufacturer Part Number (none) -> PKMCS1818E20A0-R1; Manufacturer_Name Murata Electronics -> (none); Manufacturer_Part_Number PKMCS1818E20A0-R1 -> (none); Mouser Price/Stock https://www.mouser.co.uk/ProductDetail/Murata-Electronics/P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 -> (none); Supplier Link (none) -> https://www.mouser.co.uk/ProductDetail/Murata-Electronics/P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
- R15: Manufacturer (none) -> Yageo; Manufacturer Part Number (none) -> RC0402JR-7D100KL; Manufacturer_Name Yageo -> (none); Manufacturer_Part_Number RC0402JR-7D100KL -> (none); Mouser Price/Stock https://pt.mouser.com/ProductDetail/YAGEO/RC0402JR-7D100KL?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 -> (none); Supplier Link (none) -> https://pt.mouser.com/ProductDetail/YAGEO/RC0402JR-7D100KL?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
- R16: Manufacturer (none) -> Yageo; Manufacturer Part Number (none) -> RC0402DR-07130KL; Manufacturer_Name Yageo -> (none); Manufacturer_Part_Number RC0402DR-07130KL -> (none); Mouser Price/Stock https://pt.mouser.com/ProductDetail/YAGEO/RC0402DR-07130KL?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 -> (none); Supplier Link (none) -> https://pt.mouser.com/ProductDetail/YAGEO/RC0402DR-07130KL?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
- R17: Manufacturer (none) -> Yageo; Manufacturer Part Number (none) -> RC0402FR-071M15L; Manufacturer_Name Yageo -> (none); Manufacturer_Part_Number RC0402FR-071M15L -> (none); Mouser Price/Stock https://pt.mouser.com/ProductDetail/YAGEO/RC0402FR-071M15L?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 -> (none); Supplier Link (none) -> https://pt.mouser.com/ProductDetail/YAGEO/RC0402FR-071M15L?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
- R18, R19: Manufacturer (none) -> Panasonic; Manufacturer Part Number (none) -> ERJ-S02J330X; Manufacturer_Name Panasonic -> (none); Manufacturer_Part_Number ERJ-S02J330X -> (none); Mouser Price/Stock https://pt.mouser.com/ProductDetail/Panasonic/ERJ-S02J330X?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 -> (none); Supplier Link (none) -> https://pt.mouser.com/ProductDetail/Panasonic/ERJ-S02J330X?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
- R20: Manufacturer (none) -> Yageo; Manufacturer Part Number (none) -> RC0402JR-7D1ML; Manufacturer_Name Yageo -> (none); Manufacturer_Part_Number RC0402JR-7D1ML -> (none); Mouser Price/Stock https://pt.mouser.com/ProductDetail/YAGEO/RC0402JR-7D1ML?qs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 -> (none); Supplier Link (none) -> https://pt.mouser.com/ProductDetail/YAGEO/RC0402JR-7D1ML?qs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

Commit message: EG-38 BOM fixed: Choosed the same suppliers for 4 components.
Parts:
- R20: Manufacturer Yageo -> Panasonic; Manufacturer Part Number RC0402JR-7D1ML -> ERJ-2RKD1004X; Mouser Part Number 603-RC0402JR-7D1ML -> 667-ERJ-2RKD1004X; Supplier Link https://pt.mouser.com/ProductDetail/YAGEO/RC0402JR-7D1ML?qs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 -> https://pt.mouser.com/ProductDetail/Panasonic/ERJ-2RKD1004X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
Changed lines of the file:
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@@
 			)
 		)
-		(property "Mouser Part Number" "603-RC0402JR-7D1ML"
+		(property "Mouser Part Number" "667-ERJ-2RKD1004X"
 			(at 123.19 97.79 0)
 			(effects
@@
 			)
 		)
-		(property "Supplier Link" "https://pt.mouser.com/ProductDetail/YAGEO/RC0402JR-7D1ML?qs=sGAEpiMZZMvdGkrng054t%252BT3WHYFVvJgwwPSFtsadAuv8VwIG4USFA%3D%3D"
+		(property "Supplier Link" "https://pt.mouser.com/ProductDetail/Panasonic/ERJ-2RKD1004X?qs=Ywefl8B65e6r4yb6mm%252BtoQ%3D%3D"
 			(at 123.19 97.79 0)
 			(effects
@@
 			)
 		)
-		(property "Manufacturer" "Yageo"
+		(property "Manufacturer" "Panasonic"
 			(at 123.19 97.79 0)
 			(effects
@@
 			)
 		)
-		(property "Manufacturer Part Number" "RC0402JR-7D1ML"
+		(property "Manufacturer Part Number" "ERJ-2RKD1004X"
 			(at 123.19 97.79 0)
 			(effects
