File: hardware/gateway/mcu.kicad_sch (KiCad schematic)
At the start: 31 parts, among them IC1 STM8L151K4T6, IC5 MB85RC64TAPNF-G-BDERE1, J1 G8250041000YEU, J2 M20-9770342, Q1 IRLML6402TRPBF, U1 2462

Commit message: EG-38 Replaced all BOM field names to proper ones, according with manufacturer standards.
Parts:
- C1, C2, C5, C8: Manufacturer (none) -> Yageo; Manufacturer Part Number (none) -> CC0402KRX7R7BB104; Manufacturer_Name Yageo -> (none); Manufacturer_Part_Number CC0402KRX7R7BB104 -> (none); Mouser Price/Stock https://pt.mouser.com/ProductDetail/YAGEO/CC0402KRX7R7BB104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 -> (none); Supplier Link (none) -> https://pt.mouser.com/ProductDetail/YAGEO/CC0402KRX7R7BB104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
- C3: Manufacturer (none) -> Murata; Manufacturer Part Number (none) -> GXT155R71C103KE01D; Manufacturer_Name Murata -> (none); Manufacturer_Part_Number GXT155R71C103KE01D -> (none); Mouser Price/Stock https://pt.mouser.com/ProductDetail/Murata-Electronics/GXT1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 -> (none); Supplier Link (none) -> https://pt.mouser.com/ProductDetail/Murata-Electronics/GXT1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
- C4, C7: Manufacturer (none) -> Murata; Manufacturer Part Number (none) -> GXT155R60J105KE01D; Manufacturer_Name Murata -> (none); Manufacturer_Part_Number GXT155R60J105KE01D -> (none); Mouser Price/Stock https://pt.mouser.com/ProductDetail/Murata-Electronics/GXT1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 -> (none); Supplier Link (none) -> https://pt.mouser.com/ProductDetail/Murata-Electronics/GXT1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
- C6: Manufacturer (none) -> TAYO YUDEN; Manufacturer Part Number (none) -> JMK325B7476MM-PR; Manufacturer_Name TAYO YUDEN -> (none); Manufacturer_Part_Number JMK325B7476MM-PR -> (none); Mouser Price/Stock https://pt.mouser.com/ProductDetail/TAIYO-YUDEN/JMK325B7476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 -> (none); Supplier Link (none) -> https://pt.mouser.com/ProductDetail/TAIYO-YUDEN/JMK325B7476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
- IC1: Manufacturer (none) -> STMicroelectronics; Manufacturer Part Number (none) -> STM8L151K4T6; Manufacturer_Name STMicroelectronics -> (none); Manufacturer_Part_Number STM8L151K4T6 -> (none); Mouser Price/Stock https://www.mouser.co.uk/ProductDetail/STMicroelectronics/S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 -> (none); Supplier Link (none) -> https://www.mouser.co.uk/ProductDetail/STMicroelectronics/S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
- IC5: Manufacturer (none) -> Ramxeed; Manufacturer Part Number (none) -> MB85RC64TAPNF-G-BDERE1; Manufacturer_Name Ramxeed -> (none); Manufacturer_Part_Number MB85RC64TAPNF-G-BDERE1 -> (none); Mouser Price/Stock https://www.mouser.co.uk/ProductDetail/Fujitsu-Semiconducto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 -> (none); Supplier Link (none) -> https://www.mouser.co.uk/ProductDetail/Fujitsu-Semiconducto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
- J1: Manufacturer (none) -> Amphenol; Manufacturer Part Number (none) -> G8250041000YEU; Manufacturer_Name Amphenol -> (none); Manufacturer_Part_Number G8250041000YEU -> (none); Mouser Price/Stock https://www.mouser.co.uk/ProductDetail/Amphenol-Commercial-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 -> (none); Supplier Link (none) -> https://www.mouser.co.uk/ProductDetail/Amphenol-Commercial-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
- J2: Manufacturer (none) -> Harwin; Manufacturer Part Number (none) -> M20-9770342; Manufacturer_Name Harwin -> (none); Manufacturer_Part_Number M20-9770342 -> (none); Mouser Price/Stock https://www.mouser.co.uk/ProductDetail/Harwin/M20-9770342?q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 -> (none); Supplier Link (none) -> https://www.mouser.co.uk/ProductDetail/Harwin/M20-9770342?q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
- LED1: Manufacturer (none) -> Kingbright; Manufacturer Part Number (none) -> WP710A10LVBC/D; Manufacturer_Name Kingbright -> (none); Manufacturer_Part_Number WP710A10LVBC/D -> (none); Mouser Price/Stock https://www.mouser.co.uk/ProductDetail/Kingbright/WP710A10L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 -> (none); Supplier Link (none) -> https://www.mouser.co.uk/ProductDetail/Kingbright/WP710A10L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
- LED2: Manufacturer (none) -> Vishay; Manufacturer Part Number (none) -> TLHY4400-AS12Z; Manufacturer_Name Vishay -> (none); Manufacturer_Part_Number TLHY4400-AS12Z -> (none); Mouser Price/Stock https://www.mouser.co.uk/ProductDetail/Vishay-Semiconductor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 -> (none); Supplier Link (none) -> https://www.mouser.co.uk/ProductDetail/Vishay-Semiconductor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
- LED3: Manufacturer (none) -> Vishay; Manufacturer Part Number (none) -> TLHR4400-AS12Z; Manufacturer_Name Vishay -> (none); Manufacturer_Part_Number TLHR4400-AS12Z -> (none); Mouser Price/Stock https://www.mouser.co.uk/ProductDetail/Vishay-Semiconductor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 -> (none); Supplier Link (none) -> https://www.mouser.co.uk/ProductDetail/Vishay-Semiconductor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
- Q1: Manufacturer (none) -> Infineon; Manufacturer Part Number (none) -> IRLML6402TRPBF; Manufacturer_Name Infineon -> (none); Manufacturer_Part_Number IRLML6402TRPBF -> (none); Mouser Price/Stock https://www.mouser.co.uk/ProductDetail/Infineon-Technologie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 -> (none); Supplier Link (none) -> https://www.mouser.co.uk/ProductDetail/Infineon-Technologie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
- R1, R3: Manufacturer (none) -> Yageo; Manufacturer Part Number (none) -> RC0402JR-7D100KL; Manufacturer_Name Yageo -> (none); Manufacturer_Part_Number RC0402JR-7D100KL -> (none); Mouser Price/Stock https://pt.mouser.com/ProductDetail/YAGEO/RC0402JR-7D100KL?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 -> (none); Supplier Link (none) -> https://pt.mouser.com/ProductDetail/YAGEO/RC0402JR-7D100KL?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
- R10, R9: Manufacturer (none) -> Yageo; Manufacturer Part Number (none) -> AC0402JR-0750RL; Manufacturer_Name Yageo -> (none); Manufacturer_Part_Number AC0402JR-0750RL -> (none); Mouser Price/Stock https://pt.mouser.com/ProductDetail/YAGEO/AC0402JR-0750RL?q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 -> (none); Supplier Link (none) -> https://pt.mouser.com/ProductDetail/YAGEO/AC0402JR-0750RL?q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
- R11, R12, R4: Manufacturer (none) -> Panasonic; Manufacturer Part Number (none) -> AC0402JR-7D10KL; Manufacturer_Name Panasonic -> (none); Manufacturer_Part_Number AC0402JR-7D10KL -> (none); Mouser Price/Stock https://pt.mouser.com/ProductDetail/YAGEO/AC0402JR-7D10KL?q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 -> (none); Supplier Link (none) -> https://pt.mouser.com/ProductDetail/YAGEO/AC0402JR-7D10KL?q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
- R2: Manufacturer (none) -> Yageo; Manufacturer Part Number (none) -> RC0402JR-7D1ML; Manufacturer_Name Yageo -> (none); Manufacturer_Part_Number RC0402JR-7D1ML -> (none); Mouser Price/Stock https://pt.mouser.com/ProductDetail/YAGEO/RC0402JR-7D1ML?qs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 -> (none); Supplier Link (none) -> https://pt.mouser.com/ProductDetail/YAGEO/RC0402JR-7D1ML?qs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
- R5: Manufacturer (none) -> Panasonic; Manufacturer Part Number (none) -> ERJ-2RKD1004X; Manufacturer_Name Panasonic -> (none); Manufacturer_Part_Number ERJ-2RKD1004X -> (none); Mouser Price/Stock https://pt.mouser.com/ProductDetail/Panasonic/ERJ-2RKD1004X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 -> (none); Supplier Link (none) -> https://pt.mouser.com/ProductDetail/Panasonic/ERJ-2RKD1004X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
- R6: Manufacturer (none) -> Panasonic; Manufacturer Part Number (none) -> ERJ-2RKD5103X; Manufacturer_Name Panasonic -> (none); Manufacturer_Part_Number ERJ-2RKD5103X -> (none); Mouser Price/Stock https://pt.mouser.com/ProductDetail/Panasonic/ERJ-2RKD5103X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 -> (none); Supplier Link (none) -> https://pt.mouser.com/ProductDetail/Panasonic/ERJ-2RKD5103X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
- R7: Manufacturer (none) -> Yageo; Manufacturer Part Number (none) -> RC0402JR-7D1KL; Manufacturer_Name Yageo -> (none); Manufacturer_Part_Number RC0402JR-7D1KL -> (none); Mouser Price/Stock https://pt.mouser.com/ProductDetail/YAGEO/RC0402JR-7D1KL?qs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 -> (none); Supplier Link (none) -> https://pt.mouser.com/ProductDetail/YAGEO/RC0402JR-7D1KL?qs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
- R8: Manufacturer (none) -> Yageo; Manufacturer Part Number (none) -> AC0402JR-7D100RL; Manufacturer_Name Yageo -> (none); Manufacturer_Part_Number AC0402JR-7D100RL -> (none); Mouser Price/Stock https://pt.mouser.com/ProductDetail/YAGEO/AC0402JR-7D100RL?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 -> (none); Supplier Link (none) -> https://pt.mouser.com/ProductDetail/YAGEO/AC0402JR-7D100RL?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
- S1: Manufacturer (none) -> LITTELFUSE; Manufacturer Part Number (none) -> MASM-14R-8-10; Manufacturer_Name LITTELFUSE -> (none); Manufacturer_Part_Number MASM-14R-8-10 -> (none); Mouser Price/Stock https://www.mouser.co.uk/ProductDetail/Littelfuse/MASM-14R-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 -> (none); Supplier Link (none) -> https://www.mouser.co.uk/ProductDetail/Littelfuse/MASM-14R-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
- S2: Manufacturer (none) -> E-Switch; Manufacturer Part Number (none) -> TL6120DF160QG; Manufacturer_Name E-Switch -> (none); Manufacturer_Part_Number TL6120DF160QG -> (none); Mouser Price/Stock https://www.mouser.co.uk/ProductDetail/E-Switch/TL6120DF160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 -> (none); Supplier Link (none) -> https://www.mouser.co.uk/ProductDetail/E-Switch/TL6120DF160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
- U1: Manufacturer (none) -> Keystone Electronics; Manufacturer Part Number (none) -> 2462; Manufacturer_Name Keystone Electronics -> (none); Manufacturer_Part_Number 2462 -> (none); Mouser Price/Stock https://www.mouser.co.uk/ProductDetail/Keystone-Electronics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 -> (none); Supplier Link (none) -> https://www.mouser.co.uk/ProductDetail/Keystone-Electronics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

Commit message: EG-38 BOM fixed: Choosed the same suppliers for 4 components.
Parts:
- R2: Manufacturer Yageo -> Panasonic; Manufacturer Part Number RC0402JR-7D1ML -> ERJ-2RKD1004X; Mouser Part Number 603-RC0402JR-7D1ML -> 667-ERJ-2RKD1004X; Supplier Link https://pt.mouser.com/ProductDetail/YAGEO/RC0402JR-7D1ML?qs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 -> https://pt.mouser.com/ProductDetail/Panasonic/ERJ-2RKD1004X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
Changed lines of the file:
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@@
 			)
 		)
-		(property "Mouser Part Number" "603-RC0402JR-7D1ML"
+		(property "Mouser Part Number" "667-ERJ-2RKD1004X"
 			(at 49.53 64.77 0)
 			(effects
@@
 			)
 		)
-		(property "Supplier Link" "https://pt.mouser.com/ProductDetail/YAGEO/RC0402JR-7D1ML?qs=sGAEpiMZZMvdGkrng054t%252BT3WHYFVvJgwwPSFtsadAuv8VwIG4USFA%3D%3D"
+		(property "Supplier Link" "https://pt.mouser.com/ProductDetail/Panasonic/ERJ-2RKD1004X?qs=Ywefl8B65e6r4yb6mm%252BtoQ%3D%3D"
 			(at 49.53 64.77 0)
 			(effects
@@
 			)
 		)
-		(property "Manufacturer" "Yageo"
+		(property "Manufacturer" "Panasonic"
 			(at 49.53 64.77 0)
 			(effects
@@
 			)
 		)
-		(property "Manufacturer Part Number" "RC0402JR-7D1ML"
+		(property "Manufacturer Part Number" "ERJ-2RKD1004X"
 			(at 49.53 64.77 0)
 			(effects
