File: hardware/gateway/rf.kicad_sch (KiCad schematic)
At the start: 28 parts, among them IC2 CC1101RGPR, Y1 NX3225GA-26.000M-STD-CRG-2

Commit message: EG-38 Replaced all BOM field names to proper ones, according with manufacturer standards.
Parts:
- ANT1: Manufacturer (none) -> TE Connectivity; Manufacturer Part Number (none) -> ANT-868-HETH; Manufacturer_Name TE Connectivity -> (none); Manufacturer_Part_Number ANT-868-HETH -> (none); Mouser Price/Stock https://eu.mouser.com/ProductDetail/TE-Connectivity-Linx-Te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 -> (none); Supplier Link (none) -> https://eu.mouser.com/ProductDetail/TE-Connectivity-Linx-Te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
- C10, C11, C12, C14, C15, C16, C17: Manufacturer (none) -> Yageo; Manufacturer Part Number (none) -> CC0402KRX7R7BB104; Manufacturer_Name Yageo -> (none); Manufacturer_Part_Number CC0402KRX7R7BB104 -> (none); Mouser Price/Stock https://pt.mouser.com/ProductDetail/YAGEO/CC0402KRX7R7BB104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 -> (none); Supplier Link (none) -> https://pt.mouser.com/ProductDetail/YAGEO/CC0402KRX7R7BB104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
- C121: Manufacturer (none) -> Murata; Manufacturer Part Number (none) -> GRM1555C1H1R0BA01J; Manufacturer_Name Murata -> (none); Manufacturer_Part_Number GRM1555C1H1R0BA01J -> (none); Mouser Price/Stock https://pt.mouser.com/ProductDetail/Murata-Electronics/GRM1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 -> (none); Supplier Link (none) -> https://pt.mouser.com/ProductDetail/Murata-Electronics/GRM1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
- C122, C131: Manufacturer (none) -> Murata; Manufacturer Part Number (none) -> GRM1555C1E1R5BA01D; Manufacturer_Name Murata -> (none); Manufacturer_Part_Number GRM1555C1E1R5BA01D -> (none); Mouser Price/Stock https://pt.mouser.com/ProductDetail/Murata-Electronics/GRM1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 -> (none); Supplier Link (none) -> https://pt.mouser.com/ProductDetail/Murata-Electronics/GRM1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
- C123: Manufacturer (none) -> Murata; Manufacturer Part Number (none) -> GRM1555C1H3R3WA01D; Manufacturer_Name Murata -> (none); Manufacturer_Part_Number GRM1555C1H3R3WA01D -> (none); Mouser Price/Stock https://pt.mouser.com/ProductDetail/Murata-Electronics/GRM1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 -> (none); Supplier Link (none) -> https://pt.mouser.com/ProductDetail/Murata-Electronics/GRM1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
- C124: Manufacturer (none) -> Murata; Manufacturer Part Number (none) -> GRM1555C1H101FA01J; Manufacturer_Name Murata -> (none); Manufacturer_Part_Number GRM1555C1H101FA01J -> (none); Mouser Price/Stock https://pt.mouser.com/ProductDetail/Murata-Electronics/GRM1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 -> (none); Supplier Link (none) -> https://pt.mouser.com/ProductDetail/Murata-Electronics/GRM1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
- C125: Manufacturer (none) -> Murata; Manufacturer Part Number (none) -> GRM1555C1H120FA01D; Manufacturer_Name Murata -> (none); Manufacturer_Part_Number GRM1555C1H120FA01D -> (none); Mouser Price/Stock https://pt.mouser.com/ProductDetail/Murata-Electronics/GRM1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 -> (none); Supplier Link (none) -> https://pt.mouser.com/ProductDetail/Murata-Electronics/GRM1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
- C13: Manufacturer (none) -> Murata; Manufacturer Part Number (none) -> GXT155R60J105KE01D; Manufacturer_Name Murata -> (none); Manufacturer_Part_Number GXT155R60J105KE01D -> (none); Mouser Price/Stock https://pt.mouser.com/ProductDetail/Murata-Electronics/GXT1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 -> (none); Supplier Link (none) -> https://pt.mouser.com/ProductDetail/Murata-Electronics/GXT1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
- C18, C19: Manufacturer (none) -> Kemet; Manufacturer Part Number (none) -> C0402C120F5GACAUTO; Manufacturer_Name Kemet -> (none); Manufacturer_Part_Number C0402C120F5GACAUTO -> (none); Mouser Price/Stock https://pt.mouser.com/ProductDetail/KEMET/C0402C120F5GACAUT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 -> (none); Supplier Link (none) -> https://pt.mouser.com/ProductDetail/KEMET/C0402C120F5GACAUT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
- C9: Manufacturer (none) -> TAYO YUDEN; Manufacturer Part Number (none) -> JMK325B7476MM-PR; Manufacturer_Name TAYO YUDEN -> (none); Manufacturer_Part_Number JMK325B7476MM-PR -> (none); Mouser Price/Stock https://pt.mouser.com/ProductDetail/TAIYO-YUDEN/JMK325B7476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 -> (none); Supplier Link (none) -> https://pt.mouser.com/ProductDetail/TAIYO-YUDEN/JMK325B7476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
- FB1: Manufacturer (none) -> Murata Electronics; Manufacturer Part Number (none) -> BLM18KG601SN1D; Manufacturer_Name Murata Electronics -> (none); Manufacturer_Part_Number BLM18KG601SN1D -> (none); Mouser Price/Stock https://www.mouser.co.uk/ProductDetail/Murata-Electronics/B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 -> (none); Supplier Link (none) -> https://www.mouser.co.uk/ProductDetail/Murata-Electronics/B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
- IC2: Manufacturer (none) -> Texas Instruments; Manufacturer Part Number (none) -> CC1101RGPR; Manufacturer_Name Texas Instruments -> (none); Manufacturer_Part_Number CC1101RGPR -> (none); Mouser Price/Stock https://www.mouser.co.uk/ProductDetail/Texas-Instruments/CC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 -> (none); Supplier Link (none) -> https://www.mouser.co.uk/ProductDetail/Texas-Instruments/CC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
- L121, L123, L124, L131: Manufacturer (none) -> Murata; Manufacturer Part Number (none) -> LQW15AN12NJ80D; Manufacturer_Name Murata -> (none); Manufacturer_Part_Number LQW15AN12NJ80D -> (none); Mouser Price/Stock https://pt.mouser.com/ProductDetail/Murata-Electronics/LQW1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 -> (none); Supplier Link (none) -> https://pt.mouser.com/ProductDetail/Murata-Electronics/LQW1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
- L122, L132: Manufacturer (none) -> Murata; Manufacturer Part Number (none) -> LQG15HH18NJ02D; Manufacturer_Name Murata -> (none); Manufacturer_Part_Number LQG15HH18NJ02D -> (none); Mouser Price/Stock https://pt.mouser.com/ProductDetail/Murata-Electronics/LQG1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 -> (none); Supplier Link (none) -> https://pt.mouser.com/ProductDetail/Murata-Electronics/LQG1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
- R13: Manufacturer (none) -> Panasonic; Manufacturer Part Number (none) -> ERJ-PA2F5602X; Manufacturer_Name Panasonic -> (none); Manufacturer_Part_Number ERJ-PA2F5602X -> (none); Mouser Price/Stock https://pt.mouser.com/ProductDetail/Panasonic/ERJ-PA2F5602X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 -> (none); Supplier Link (none) -> https://pt.mouser.com/ProductDetail/Panasonic/ERJ-PA2F5602X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
- Y1: Manufacturer (none) -> NDK; Manufacturer Part Number (none) -> NX3225GA-26.000M-STD-CRG-2; Manufacturer_Name NDK -> (none); Manufacturer_Part_Number NX3225GA-26.000M-STD-CRG-2 -> (none); Mouser Price/Stock https://www.mouser.co.uk/ProductDetail/NDK/NX3225GA-26.000M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 -> (none); Supplier Link (none) -> https://www.mouser.co.uk/ProductDetail/NDK/NX3225GA-26.000M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

Commit message: EG-38 BOM fixed: Choosed the same suppliers for 4 components.
Parts:
- C18, C19: Manufacturer Kemet -> Murata Electronics; Manufacturer Part Number C0402C120F5GACAUTO -> GRM1555C1H120FA1D; Mouser Part Number 80-C0402C120F5GAUTO -> 81-GRM1555C1H120FA1D; Supplier Link https://pt.mouser.com/ProductDetail/KEMET/C0402C120F5GACAUT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 -> https://pt.mouser.com/ProductDetail/Murata-Electronics/GRM1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
Changed lines of the file:
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@@
 			)
 		)
-		(property "Mouser Part Number" "80-C0402C120F5GAUTO"
+		(property "Mouser Part Number" "81-GRM1555C1H120FA1D"
 			(at 133.35 140.97 0)
 			(effects
@@
 			)
 		)
-		(property "Supplier Link" "https://pt.mouser.com/ProductDetail/KEMET/C0402C120F5GACAUTO?qs=rrS6PyfT74fKM3c0c1DHjw%3D%3D"
+		(property "Supplier Link" "https://pt.mouser.com/ProductDetail/Murata-Electronics/GRM1555C1H120FA01D?qs=ouTquLLW2S4GiX6b03cbUg%3D%3D"
 			(at 133.35 140.97 0)
 			(effects
@@
 			)
 		)
-		(property "Manufacturer" "Kemet"
+		(property "Manufacturer" "Murata Electronics"
 			(at 133.35 140.97 0)
 			(effects
@@
 			)
 		)
-		(property "Manufacturer Part Number" "C0402C120F5GACAUTO"
+		(property "Manufacturer Part Number" "GRM1555C1H120FA1D"
 			(at 133.35 140.97 0)
 			(effects
@@
 			)
 		)
-		(property "Mouser Part Number" "80-C0402C120F5GAUTO"
+		(property "Mouser Part Number" "81-GRM1555C1H120FA1D"
 			(at 69.85 140.97 0)
 			(effects
@@
 			)
 		)
-		(property "Supplier Link" "https://pt.mouser.com/ProductDetail/KEMET/C0402C120F5GACAUTO?qs=rrS6PyfT74fKM3c0c1DHjw%3D%3D"
+		(property "Supplier Link" "https://pt.mouser.com/ProductDetail/Murata-Electronics/GRM1555C1H120FA01D?qs=ouTquLLW2S4GiX6b03cbUg%3D%3D"
 			(at 69.85 140.97 0)
 			(effects
@@
 			)
 		)
-		(property "Manufacturer" "Kemet"
+		(property "Manufacturer" "Murata Electronics"
 			(at 69.85 140.97 0)
 			(effects
@@
 			)
 		)
-		(property "Manufacturer Part Number" "C0402C120F5GACAUTO"
+		(property "Manufacturer Part Number" "GRM1555C1H120FA1D"
 			(at 69.85 140.97 0)
 			(effects
