File: hardware/sensor/sensor.kicad_sch (KiCad schematic)
At the start: 36 parts, among them IC1 STM8L001J3M3, IC2 Si4012-C1001GTR, IC3 TPS3839L30DBZR, J1 M20-9770342

Commit message: EG-37 BOM and gerbers generated due to components replacement.
Parts:
- H1: Manufacturer (none) -> TE Connectivity; Manufacturer Part Number (none) -> BAT-HLD-006-SMT; Manufacturer_Name TE Connectivity -> (none); Manufacturer_Part_Number BAT-HLD-006-SMT -> (none); Mouser Price/Stock https://www.mouser.co.uk/ProductDetail/TE-Connectivity-Linx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 -> (none); Supplier Link (none) -> https://www.mouser.co.uk/ProductDetail/TE-Connectivity-Linx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
Changed lines of the file:
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@@
 			)
 		)
-		(property "Mouser Price/Stock" "https://www.mouser.co.uk/ProductDetail/TE-Connectivity-Linx-Technologies/BAT-HLD-006-SMT?qs=TuK3vfAjtkUyTQHMSqIP6A%3D%3D"
+		(property "Supplier Link" "https://www.mouser.co.uk/ProductDetail/TE-Connectivity-Linx-Technologies/BAT-HLD-006-SMT?qs=TuK3vfAjtkUyTQHMSqIP6A%3D%3D"
 			(at 22.86 -558.09 0)
 			(effects
@@
 			)
 		)
-		(property "Manufacturer_Name" "TE Connectivity"
+		(property "Manufacturer" "TE Connectivity"
 			(at 22.86 -658.09 0)
 			(effects
@@
 			)
 		)
-		(property "Manufacturer_Part_Number" "BAT-HLD-006-SMT"
+		(property "Manufacturer Part Number" "BAT-HLD-006-SMT"
 			(at 22.86 -758.09 0)
 			(effects

Commit message: EG-37 Gerbers, BOM and CPL reviewed.
Parts:
- ANT1: Manufacturer (none) -> TE Connectivity; Manufacturer Part Number (none) -> ANT-868-HETH; Manufacturer_Name TE Connectivity -> (none); Manufacturer_Part_Number ANT-868-HETH -> (none); Mouser Price/Stock https://pt.mouser.com/ProductDetail/TE-Connectivity-Linx-Te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 -> (none); Supplier Link (none) -> https://pt.mouser.com/ProductDetail/TE-Connectivity-Linx-Te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
- C1, C2, C4: Manufacturer (none) -> Murata Electronics; Manufacturer Part Number (none) -> GCJ188R72A104KA1D; Manufacturer_Name Murata -> (none); Manufacturer_Part_Number GCJ188R72A104KA1D -> (none); Mouser Price/Stock https://pt.mouser.com/ProductDetail/Murata-Electronics/GCJ1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 -> (none); Supplier Link (none) -> https://pt.mouser.com/ProductDetail/Murata-Electronics/GCJ1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
- C3, C6: Manufacturer (none) -> TAYO YUDEN; Manufacturer Part Number (none) -> MBASE168SB7105KTNA18; Manufacturer_Name TAYO YUDEN -> (none); Manufacturer_Part_Number MBASE168SB7105KTNA18 -> (none); Mouser Price/Stock https://pt.mouser.com/ProductDetail/TAIYO-YUDEN/MBASE168SB7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 -> (none); Supplier Link (none) -> https://pt.mouser.com/ProductDetail/TAIYO-YUDEN/MBASE168SB7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
- C5, C8: Manufacturer (none) -> TAYO YUDEN; Manufacturer Part Number (none) -> JMK325B7476MM-PR; Manufacturer_Name TAYO YUDEN -> (none); Manufacturer_Part_Number JMK325B7476MM-PR -> (none); Mouser Price/Stock https://pt.mouser.com/ProductDetail/TAIYO-YUDEN/JMK325B7476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 -> (none); Supplier Link (none) -> https://pt.mouser.com/ProductDetail/TAIYO-YUDEN/JMK325B7476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
- C7: Manufacturer (none) -> Vishay; Manufacturer Part Number (none) -> VJ0603Y101MXQCW1BC; Manufacturer_Name Vishay -> (none); Manufacturer_Part_Number VJ0603Y101MXQCW1BC -> (none); Mouser Price/Stock https://pt.mouser.com/ProductDetail/Vishay-Vitramon/VJ0603Y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 -> (none); Supplier Link (none) -> https://pt.mouser.com/ProductDetail/Vishay-Vitramon/VJ0603Y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
- CC1: Manufacturer (none) -> Murata Electronics; Manufacturer Part Number (none) -> GRM1555C1H680FA01J; Manufacturer_Name Murata -> (none); Manufacturer_Part_Number GRM1555C1H680FA01J -> (none); Mouser Price/Stock https://eu.mouser.com/ProductDetail/Murata-Electronics/GRM1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 -> (none); Supplier Link (none) -> https://eu.mouser.com/ProductDetail/Murata-Electronics/GRM1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
- CM1, CM3: Manufacturer (none) -> Murata Electronics; Manufacturer Part Number (none) -> GRM1555C1H2R4WA01D; Manufacturer_Name Murata -> (none); Manufacturer_Part_Number GRM1555C1H2R4WA01D -> (none); Mouser Price/Stock https://eu.mouser.com/ProductDetail/Murata-Electronics/GRM1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 -> (none); Supplier Link (none) -> https://eu.mouser.com/ProductDetail/Murata-Electronics/GRM1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
- CM2: Manufacturer (none) -> Kyocera; Manufacturer Part Number (none) -> 04025A1R2DAT2A; Manufacturer_Name Kyocera -> (none); Manufacturer_Part_Number 04025A1R2DAT2A -> (none); Mouser Price/Stock https://pt.mouser.com/ProductDetail/KYOCERA-AVX/04025A1R2DA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 -> (none); Supplier Link (none) -> https://pt.mouser.com/ProductDetail/KYOCERA-AVX/04025A1R2DA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
- CM5, CM6: Manufacturer (none) -> Murata Electronics; Manufacturer Part Number (none) -> GCQ1555C1H5R1WB01D; Manufacturer_Name Murata -> (none); Manufacturer_Part_Number GCQ1555C1H5R1WB01D -> (none); Mouser Price/Stock https://pt.mouser.com/ProductDetail/Murata-Electronics/GCQ1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 -> (none); Supplier Link (none) -> https://pt.mouser.com/ProductDetail/Murata-Electronics/GCQ1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
- FB1: Manufacturer (none) -> Murata Electronics; Manufacturer Part Number (none) -> BLM18KG601SN1D; Manufacturer_Name Murata Electronics -> (none); Manufacturer_Part_Number BLM18KG601SN1D -> (none); Mouser Price/Stock https://pt.mouser.com/ProductDetail/Murata-Electronics/BLM1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 -> (none); Supplier Link (none) -> https://pt.mouser.com/ProductDetail/Murata-Electronics/BLM1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
- IC1: Manufacturer (none) -> STMicroelectronics; Manufacturer Part Number (none) -> STM8L001J3M3; Manufacturer_Name STMicroelectronics -> (none); Manufacturer_Part_Number STM8L001J3M3 -> (none); Mouser Price/Stock https://www.mouser.co.uk/ProductDetail/STMicroelectronics/S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 -> (none); Supplier Link (none) -> https://www.mouser.co.uk/ProductDetail/STMicroelectronics/S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
- IC2: Manufacturer (none) -> Silicon Labs; Manufacturer Part Number (none) -> Si4012-C1001GTR; Manufacturer_Name Silicon Labs -> (none); Manufacturer_Part_Number Si4012-C1001GTR -> (none); Mouser Price/Stock https://pt.mouser.com/ProductDetail/Silicon-Labs/SI4012-C10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 -> (none); Supplier Link (none) -> https://pt.mouser.com/ProductDetail/Silicon-Labs/SI4012-C10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
- IC3: Manufacturer (none) -> Texas Instruments; Manufacturer Part Number (none) -> TPS3839L30DBZR; Manufacturer_Name Texas Instruments -> (none); Manufacturer_Part_Number TPS3839L30DBZR -> (none); Mouser Price/Stock https://pt.mouser.com/ProductDetail/Texas-Instruments/TPS38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 -> (none); Supplier Link (none) -> https://pt.mouser.com/ProductDetail/Texas-Instruments/TPS38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
- J1: Manufacturer (none) -> Harwin; Manufacturer Part Number (none) -> M20-9770342; Manufacturer_Name Harwin -> (none); Manufacturer_Part_Number M20-9770342 -> (none); Mouser Price/Stock https://www.mouser.co.uk/ProductDetail/Harwin/M20-9770342?q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 -> (none); Supplier Link (none) -> https://www.mouser.co.uk/ProductDetail/Harwin/M20-9770342?q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
- LM1: Manufacturer (none) -> Coilcraf; Manufacturer Part Number (none) -> 994-0603DC-R12XJRW; Manufacturer_Name Coilcraf -> (none); Manufacturer_Part_Number 994-0603DC-R12XJRW -> (none); Mouser Price/Stock https://eu.mouser.com/ProductDetail/Coilcraft/0603DC-R12XJR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 -> (none); Supplier Link (none) -> https://eu.mouser.com/ProductDetail/Coilcraft/0603DC-R12XJR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
- LM2, LM4: Manufacturer (none) -> Coilcraft; Manufacturer Part Number (none) -> 0402HP-3N6XGRW; Manufacturer_Name Coilcraft -> (none); Manufacturer_Part_Number 0402HP-3N6XGRW -> (none); Mouser Price/Stock https://eu.mouser.com/ProductDetail/Coilcraft/0402HP-3N6XGR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 -> (none); Supplier Link (none) -> https://eu.mouser.com/ProductDetail/Coilcraft/0402HP-3N6XGR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
- LM3: Manufacturer (none) -> Coilcraft; Manufacturer Part Number (none) -> 0402HP-30NXJRW; Manufacturer_Name Coilcraft -> (none); Manufacturer_Part_Number 0402HP-30NXJRW -> (none); Mouser Price/Stock https://eu.mouser.com/ProductDetail/Coilcraft/0402HP-30NXJR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 -> (none); Supplier Link (none) -> https://eu.mouser.com/ProductDetail/Coilcraft/0402HP-30NXJR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
- LM5: Manufacturer (none) -> Coilcraft; Manufacturer Part Number (none) -> 0402HP-6N8XGRW; Manufacturer_Name Coilcraft -> (none); Manufacturer_Part_Number 0402HP-6N8XGRW -> (none); Mouser Price/Stock https://eu.mouser.com/ProductDetail/Coilcraft/0402HP-6N8XGR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 -> (none); Supplier Link (none) -> https://eu.mouser.com/ProductDetail/Coilcraft/0402HP-6N8XGR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
- R1: Manufacturer (none) -> Rohm; Manufacturer Part Number (none) -> SFR03EZPJ105; Manufacturer_Name Rohm -> (none); Manufacturer_Part_Number SFR03EZPJ105 -> (none); Mouser Price/Stock https://pt.mouser.com/ProductDetail/ROHM-Semiconductor/SFR0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 -> (none); Supplier Link (none) -> https://pt.mouser.com/ProductDetail/ROHM-Semiconductor/SFR0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
- R2, R5: Manufacturer (none) -> Vishay; Manufacturer Part Number (none) -> RCA0603100KJNEA; Manufacturer_Name Vishay -> (none); Manufacturer_Part_Number RCA0603100KJNEA -> (none); Mouser Price/Stock https://pt.mouser.com/ProductDetail/Vishay-Draloric/RCA0603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 -> (none); Supplier Link (none) -> https://pt.mouser.com/ProductDetail/Vishay-Draloric/RCA0603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
- R3, R4: Manufacturer (none) -> Yageo; Manufacturer Part Number (none) -> AC0603JR-7W10KL; Manufacturer_Name Yageo -> (none); Manufacturer_Part_Number AC0603JR-7W10KL -> (none); Mouser Price/Stock https://pt.mouser.com/ProductDetail/YAGEO/AC0603JR-7W10KL?q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 -> (none); Supplier Link (none) -> https://pt.mouser.com/ProductDetail/YAGEO/AC0603JR-7W10KL?q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
- S1: Manufacturer (none) -> LITTELFUSE; Manufacturer Part Number (none) -> MASM-14R-8-10; Manufacturer_Name LITTELFUSE -> (none); Manufacturer_Part_Number MASM-14R-8-10 -> (none); Mouser Price/Stock https://pt.mouser.com/ProductDetail/Littelfuse/MASM-14R-8-1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 -> (none); Supplier Link (none) -> https://pt.mouser.com/ProductDetail/Littelfuse/MASM-14R-8-1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
