File: hardware/gateway/rev1/mcu_rev1.kicad_sch (KiCad schematic)
At the start: 31 parts, among them IC1 STM8L151K4T6, IC5 MB85RC64TAPNF-G-BDERE1, J1 G8250041000YEU, J2 M20-9770342, Q1 IRLML6402TRPBF, U1 2462

Commit message: Replaced 0402  by 0603 package where was possible.
Parts:
- C1, C2, C5: footprint Capacitor_SMD:C_0402_1005Metric -> Capacitor_SMD:C_0603_1608Metric; Manufacturer Yageo -> Taiyo Yuden; Manufacturer Part Number CC0402KRX7R7BB104 -> MAJCH168BB7104KT; Mouser Part Number 603-CC402KRX7R7BB104 -> 963-MAJCH168BB7104KT; Supplier Link https://pt.mouser.com/ProductDetail/YAGEO/CC0402KRX7R7BB104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 -> https://pt.mouser.com/ProductDetail/TAIYO-YUDEN/MAJCH168BB7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
- C4: footprint Capacitor_SMD:C_0402_1005Metric -> Capacitor_SMD:C_0603_1608Metric; Manufacturer Murata -> Yageo; Manufacturer Part Number GXT155R60J105KE01D -> CC603KRX5R6BB105; Mouser Part Number 81-GXT155R60J105KE1D -> 603-CC603KRX5R6BB105; Supplier Link https://pt.mouser.com/ProductDetail/Murata-Electronics/GXT1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 -> https://pt.mouser.com/ProductDetail/YAGEO/CC0603KRX5R6BB105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
- R1, R3: footprint Resistor_SMD:R_0402_1005Metric -> Resistor_SMD:R_0603_1608Metric; Manufacturer Yageo -> Vishay; Manufacturer Part Number RC0402JR-7D100KL -> MCT06030C1003FP5; Mouser Part Number 603-RC0402JR-7D100KL -> 594-MCT06030C1003FP5; Supplier Link https://pt.mouser.com/ProductDetail/YAGEO/RC0402JR-7D100KL?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 -> https://pt.mouser.com/ProductDetail/Vishay-Beyschlag/MCT060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
- R10, R9: value 50 -> 47; footprint Resistor_SMD:R_0402_1005Metric -> Resistor_SMD:R_0603_1608Metric; Manufacturer Yageo -> Panasonic; Manufacturer Part Number AC0402JR-0750RL -> ERJ-S03J470V; Mouser Part Number 603-AC0402JR-0750RL -> 667-ERJ-S03J470V; Supplier Link https://pt.mouser.com/ProductDetail/YAGEO/AC0402JR-0750RL?q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 -> https://pt.mouser.com/ProductDetail/Panasonic/ERJ-S03J470V?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
- R11, R12, R4: footprint Resistor_SMD:R_0402_1005Metric -> Resistor_SMD:R_0603_1608Metric; Manufacturer Panasonic -> Vishay; Manufacturer Part Number AC0402JR-7D10KL -> RCA060310K0JNEA; Mouser Part Number 603-AC0402JR-7D10KL -> 71-RCA060310K0JNEA; Supplier Link https://pt.mouser.com/ProductDetail/YAGEO/AC0402JR-7D10KL?q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 -> https://pt.mouser.com/ProductDetail/Vishay-Draloric/RCA0603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
- R2, R5: footprint Resistor_SMD:R_0402_1005Metric -> Resistor_SMD:R_0603_1608Metric; Manufacturer Panasonic -> Yageo; Manufacturer Part Number ERJ-2RKD1004X -> AR0603FR-071ML; Mouser Part Number 667-ERJ-2RKD1004X -> 603-AR0603FR-071ML; Supplier Link https://pt.mouser.com/ProductDetail/Panasonic/ERJ-2RKD1004X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 -> https://pt.mouser.com/ProductDetail/YAGEO/AR0603FR-071ML?qs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
- R6: footprint Resistor_SMD:R_0402_1005Metric -> Resistor_SMD:R_0603_1608Metric; Manufacturer Panasonic -> Vishay; Manufacturer Part Number ERJ-2RKD5103X -> CRCW0603-510K; Mouser Part Number 667-ERJ-2RKD5103X -> 71-CRCW0603-510K; Supplier Link https://pt.mouser.com/ProductDetail/Panasonic/ERJ-2RKD5103X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 -> https://pt.mouser.com/ProductDetail/Vishay/CRCW0603510KFKTA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
- R7: footprint Resistor_SMD:R_0402_1005Metric -> Resistor_SMD:R_0603_1608Metric; Manufacturer Part Number RC0402JR-7D1KL -> SR0603JR-071KL; Mouser Part Number 603-RC0402JR-7D1KL -> 603-SR0603JR-071KL; Supplier Link https://pt.mouser.com/ProductDetail/YAGEO/RC0402JR-7D1KL?qs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 -> https://pt.mouser.com/ProductDetail/YAGEO/SR0603JR-071KL?qs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
- R8: footprint Resistor_SMD:R_0402_1005Metric -> Resistor_SMD:R_0603_1608Metric; Manufacturer Yageo -> Vishay; Manufacturer Part Number AC0402JR-7D100RL -> CRCW0603100RJNEBC; Mouser Part Number 603-AC0402JR-7D100RL -> 71-CRCW0603100RJNEBC; Supplier Link https://pt.mouser.com/ProductDetail/YAGEO/AC0402JR-7D100RL?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 -> https://pt.mouser.com/ProductDetail/Vishay/CRCW0603100RJNEB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

Commit message: BOM fixed and finance updated
Parts:
- C6: Manufacturer Part Number JMK325B7476MM-PR -> JMK316BJ476MD-T; Mouser Part Number 963-JMK325B7476MM-PR -> 963-JMK316BJ476MD-T; Supplier Link https://pt.mouser.com/ProductDetail/TAIYO-YUDEN/JMK325B7476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 -> https://pt.mouser.com/ProductDetail/TAIYO-YUDEN/JMK316BJ476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
