File: hardware/sensor/rev1/rf_rev1.kicad_sch (KiCad schematic)
At the start: 27 parts, among them IC2 CC1101RGPR, Y1 NX3225GA-26.000M-STD-CRG-2

Commit message: EG-49 Removed a bulk capacitor.
Parts:
- removed C13: 1uF, Capacitor_SMD:C_0402_1005Metric, symbol Device:C
Changed lines of the file:
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@@
 	)
 	(junction
-		(at 121.92 33.02)
-		(diameter 0)
-		(color 0 0 0 0)
-	)
-	(junction
 		(at 163.83 86.36)
 		(diameter 0)
@@
 	(wire
 		(pts
-			(xy 130.81 33.02) (xy 121.92 33.02)
-		)
-		(stroke
-			(width 0)
-			(type default)
-		)
-	)
-	(wire
-		(pts
 			(xy 92.71 45.72) (xy 97.79 45.72)
 		)
@@
 	(wire
 		(pts
-			(xy 130.81 44.45) (xy 130.81 49.53)
-		)
-		(stroke
-			(width 0)
-			(type default)
-		)
-	)
-	(wire
-		(pts
 			(xy 121.92 114.3) (xy 148.59 114.3)
 		)
@@
 	(wire
 		(pts
-			(xy 121.92 27.94) (xy 121.92 33.02)
+			(xy 121.92 27.94) (xy 121.92 54.61)
 		)
 		(stroke
@@
 	(wire
 		(pts
-			(xy 121.92 33.02) (xy 121.92 54.61)
-		)
-		(stroke
-			(width 0)
-			(type default)
-		)
-	)
-	(wire
-		(pts
 			(xy 161.29 76.2) (xy 165.1 76.2)
 		)
@@
 	(wire
 		(pts
-			(xy 130.81 36.83) (xy 130.81 33.02)
-		)
-		(stroke
-			(width 0)
-			(type default)
-		)
-	)
-	(wire
-		(pts
 			(xy 161.29 86.36) (xy 161.29 85.09)
 		)
@@
 	)
 	(symbol
-		(lib_id "power:GND")
-		(at 130.81 49.53 0)
-		(unit 1)
-		(exclude_from_sim no)
-		(in_bom yes)
-		(on_board yes)
-		(dnp no)
-		(fields_autoplaced yes)
-		(property "Reference" "#PWR049"
-			(at 130.81 55.88 0)
-			(effects
-				(font
-					(size 1.27 1.27)
-				)
-				(hide yes)
-			)
-		)
-		(property "Value" "GND"
-			(at 130.81 54.61 0)
-			(effects
-				(font
-					(size 1.27 1.27)
-				)
-			)
-		)
-		(property "Footprint" ""
-			(at 130.81 49.53 0)
-			(effects
-				(font
-					(size 1.27 1.27)
-				)
-				(hide yes)
-			)
-		)
-		(property "Datasheet" ""
-			(at 130.81 49.53 0)
-			(effects
-				(font
-					(size 1.27 1.27)
-				)
-				(hide yes)
-			)
-		)
-		(property "Description" "Power symbol creates a global label with name \"GND\" , ground"
-			(at 130.81 49.53 0)
-			(effects
-				(font
-					(size 1.27 1.27)
-				)
-				(hide yes)
-			)
-		)
-		(pin "1"
-		)
-		(instances
-			(project "rf_rev1"
-				(path "/50a12035-955f-49d8-a6b8-24fcd6d450af"
-					(reference "#PWR?")
-					(unit 1)
-				)
-			)
-			(project "sensor_rev1"
-				(path "/d3cb7130-decc-418b-958e-e5d84a8d867f/af07603d-259f-481d-be2c-d925e27835a3"
-					(reference "#PWR049")
-					(unit 1)
-				)
-			)
-		)
-	)
-	(symbol
 		(lib_id "CC1101RGPR:CC1101RGPR")
 		(at 80.01 74.93 0)
@@
 					(unit 1)
 				)
-			)
-		)
-	)
-	(symbol
-		(lib_id "Device:C")
-		(at 130.81 40.64 0)
-		(unit 1)
-		(exclude_from_sim no)
-		(in_bom yes)
-		(on_board yes)
-		(dnp no)
-		(fields_autoplaced yes)
-		(property "Reference" "C13"
-			(at 134.62 39.3699 0)
-			(effects
-				(font
-					(size 1.27 1.27)
-				)
-				(justify left)
-			)
-		)
-		(property "Value" "1uF"
-			(at 134.62 41.9099 0)
-			(effects
-				(font
-					(size 1.27 1.27)
-				)
-				(justify left)
-			)
-		)
-		(property "Footprint" "Capacitor_SMD:C_0402_1005Metric"
-			(at 131.7752 44.45 0)
-			(effects
-				(font
-					(size 1.27 1.27)
-				)
-				(hide yes)
-			)
-		)
-		(property "Datasheet" "~"
-			(at 130.81 40.64 0)
-			(effects
-				(font
-					(size 1.27 1.27)
-				)
-				(hide yes)
-			)
-		)
-		(property "Description" "Unpolarized capacitor"
-			(at 130.81 40.64 0)
-			(effects
-				(font
-					(size 1.27 1.27)
-				)
-				(hide yes)
-			)
-		)
-		(property "Mouser Part Number" "81-GXT155R60J105KE1D"
-			(at 130.81 40.64 0)
-			(effects
-				(font
-					(size 1.27 1.27)
-				)
-				(hide yes)
-			)
-		)
-		(property "Supplier Link" "https://pt.mouser.com/ProductDetail/Murata-Electronics/GXT155R60J105KE01D?qs=d0WKAl%252BL4Kb4JfV7cPss8A%3D%3D"
-			(at 130.81 40.64 0)
-			(effects
-				(font
-					(size 1.27 1.27)
-				)
-				(hide yes)
-			)
-		)
-		(property "Manufacturer" "Murata"
-			(at 130.81 40.64 0)
-			(effects
-				(font
-					(size 1.27 1.27)
-				)
-				(hide yes)
-			)
-		)
-		(property "Manufacturer Part Number" "GXT155R60J105KE01D "
-			(at 130.81 40.64 0)
-			(effects
-				(font
-					(size 1.27 1.27)
-				)
-				(hide yes)
-			)
-		)
-		(pin "2"
-		)
-		(pin "1"
-		)
-		(instances
-			(project "rf_rev1"
-				(path "/50a12035-955f-49d8-a6b8-24fcd6d450af"
-					(reference "C?")
-					(unit 1)
-				)
-			)
-			(project "sensor_rev1"
-				(path "/d3cb7130-decc-418b-958e-e5d84a8d867f/af07603d-259f-481d-be2c-d925e27835a3"
-					(reference "C13")
-					(unit 1)
-				)

Commit message: EG-49 All components reviewed, MCU and RF.
Parts:
- removed C7: GRM31CR61A107MEA8L, GRM31x, symbol GRM31CR61A107MEA8L:GRM31CR61A107MEA8L
- Y1: Supplier Link https://www.mouser.co.uk/ProductDetail/NDK/NX3225GA-26.000M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 -> https://www.mouser.co.uk/en/ProductDetail/NDK/STDCRG2-26M?q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
- renumbered C16 to C10, C19 to C101, C17 to C11, C12 to C5, C11 to C51, C14 to C6, C10 to C7, C18 to C81, C15 to C9, R13 to R171

Commit message: EG-49 All  components parameters standardized for mouser.
Parts:
- C10, C11, C5, C51, C6, C7, C9: Manufacturer Yageo -> (none); Manufacturer Part Number CC0402KRX7R7BB104 -> (none); Manufacturer_Name (none) -> Yageo; Manufacturer_Part_Number (none) -> CC0402KRX7R7BB104; Mouser Price/Stock (none) -> https://pt.mouser.com/ProductDetail/YAGEO/CC0402KRX7R7BB104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; Supplier Link https://pt.mouser.com/ProductDetail/YAGEO/CC0402KRX7R7BB104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 -> (none)
- C101, C81: Manufacturer Murata Electronics -> (none); Manufacturer Part Number GRM1555C1H120FA1D -> (none); Manufacturer_Name (none) -> Murata Electronics; Manufacturer_Part_Number (none) -> GRM1555C1H120FA1D; Mouser Price/Stock (none) -> https://pt.mouser.com/ProductDetail/Murata-Electronics/GRM1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; Supplier Link https://pt.mouser.com/ProductDetail/Murata-Electronics/GRM1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 -> (none)
- C121: Manufacturer Murata -> (none); Manufacturer Part Number GRM1555C1H1R0BA01J -> (none); Manufacturer_Name (none) -> Murata; Manufacturer_Part_Number (none) -> GRM1555C1H1R0BA01J; Mouser Price/Stock (none) -> https://pt.mouser.com/ProductDetail/Murata-Electronics/GRM1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; Supplier Link https://pt.mouser.com/ProductDetail/Murata-Electronics/GRM1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 -> (none)
- C122, C131: Manufacturer Murata -> (none); Manufacturer Part Number GRM1555C1E1R5BA01D -> (none); Manufacturer_Name (none) -> Murata; Manufacturer_Part_Number (none) -> GRM1555C1E1R5BA01D; Mouser Price/Stock (none) -> https://pt.mouser.com/ProductDetail/Murata-Electronics/GRM1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; Supplier Link https://pt.mouser.com/ProductDetail/Murata-Electronics/GRM1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 -> (none)
- C123: Manufacturer Murata -> (none); Manufacturer Part Number GRM1555C1H3R3WA01D -> (none); Manufacturer_Name (none) -> Murata; Manufacturer_Part_Number (none) -> GRM1555C1H3R3WA01D; Mouser Price/Stock (none) -> https://pt.mouser.com/ProductDetail/Murata-Electronics/GRM1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; Supplier Link https://pt.mouser.com/ProductDetail/Murata-Electronics/GRM1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 -> (none)
- C124: Manufacturer Murata -> (none); Manufacturer Part Number GRM1555C1H101FA01J -> (none); Manufacturer_Name (none) -> Murata; Manufacturer_Part_Number (none) -> GRM1555C1H101FA01J; Mouser Price/Stock (none) -> https://pt.mouser.com/ProductDetail/Murata-Electronics/GRM1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; Supplier Link https://pt.mouser.com/ProductDetail/Murata-Electronics/GRM1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 -> (none)
- C125: Manufacturer Murata -> (none); Manufacturer Part Number GRM1555C1H120FA01D -> (none); Manufacturer_Name (none) -> Murata; Manufacturer_Part_Number (none) -> GRM1555C1H120FA01D; Mouser Price/Stock (none) -> https://pt.mouser.com/ProductDetail/Murata-Electronics/GRM1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; Supplier Link https://pt.mouser.com/ProductDetail/Murata-Electronics/GRM1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 -> (none)
- FB1: Manufacturer Murata Electronics -> (none); Manufacturer Part Number BLM18KG601SN1D -> (none); Manufacturer_Name (none) -> Murata Electronics; Manufacturer_Part_Number (none) -> BLM18KG601SN1D; Mouser Price/Stock (none) -> https://www.mouser.co.uk/ProductDetail/Murata-Electronics/B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; Supplier Link https://www.mouser.co.uk/ProductDetail/Murata-Electronics/B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 -> (none)
- IC2: Manufacturer Texas Instruments -> (none); Manufacturer Part Number CC1101RGPR -> (none); Manufacturer_Name (none) -> Texas Instruments; Manufacturer_Part_Number (none) -> CC1101RGPR; Mouser Price/Stock (none) -> https://www.mouser.co.uk/ProductDetail/Texas-Instruments/CC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; Supplier Link https://www.mouser.co.uk/ProductDetail/Texas-Instruments/CC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 -> (none)
- L121, L123, L124, L131: Manufacturer Murata -> (none); Manufacturer Part Number LQW15AN12NJ80D -> (none); Manufacturer_Name (none) -> Murata; Manufacturer_Part_Number (none) -> LQW15AN12NJ80D; Mouser Price/Stock (none) -> https://pt.mouser.com/ProductDetail/Murata-Electronics/LQW1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; Supplier Link https://pt.mouser.com/ProductDetail/Murata-Electronics/LQW1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 -> (none)
- L122, L132: Manufacturer Murata -> (none); Manufacturer Part Number LQG15HH18NJ02D -> (none); Manufacturer_Name (none) -> Murata; Manufacturer_Part_Number (none) -> LQG15HH18NJ02D; Mouser Price/Stock (none) -> https://pt.mouser.com/ProductDetail/Murata-Electronics/LQG1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; Supplier Link https://pt.mouser.com/ProductDetail/Murata-Electronics/LQG1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 -> (none)
- R171: Manufacturer Panasonic -> (none); Manufacturer Part Number ERJ-PA2F5602X -> (none); Manufacturer_Name (none) -> Panasonic; Manufacturer_Part_Number (none) -> ERJ-PA2F5602X; Mouser Price/Stock (none) -> https://pt.mouser.com/ProductDetail/Panasonic/ERJ-PA2F5602X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; Supplier Link https://pt.mouser.com/ProductDetail/Panasonic/ERJ-PA2F5602X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 -> (none)
- Y1: Manufacturer NDK -> (none); Manufacturer Part Number NX3225GA-26.000M-STD-CRG-2 -> (none); Manufacturer_Name (none) -> NDK; Manufacturer_Part_Number (none) -> NX3225GA-26.000M-STD-CRG-2; Mouser Price/Stock (none) -> https://www.mouser.co.uk/en/ProductDetail/NDK/STDCRG2-26M?q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; Supplier Link https://www.mouser.co.uk/en/ProductDetail/NDK/STDCRG2-26M?q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 -> (none)

Commit message: EG-49 Antenna hole placed.
Parts:
- added ANT1: ~, MyParts:Antenna_hole, symbol antenna_hole:Antenna_Hole
Connections:
- net at C125.2: now also ANT1.1 (ANT)
Changed lines of the file:
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@@
+	(wire
+		(pts
+			(xy 217.17 81.28) (xy 220.98 81.28)
+		)
+		(stroke
+			(width 0)
+			(type default)
+		)
+	)
 	(wire
 		(pts
@@
 					(unit 1)
 				)
+			)
+		)
+	)
+	(symbol
+		(lib_id "antenna_hole:Antenna_Hole")
+		(at 226.06 81.28 180)
+		(unit 1)
+		(exclude_from_sim no)
+		(in_bom yes)
+		(on_board yes)
+		(dnp no)
+		(fields_autoplaced yes)
+		(property "Reference" "ANT1"
+			(at 229.87 80.0099 0)
+			(effects
+				(font
+					(size 1.27 1.27)
+				)
+				(justify right)
+			)
+		)
+		(property "Value" "~"
+			(at 229.87 82.5499 0)
+			(effects
+				(font
+					(size 1.27 1.27)
+				)
+				(justify right)
+			)
+		)
+		(property "Footprint" "MyParts:Antenna_hole"
+			(at 226.06 81.28 0)
+			(effects
+				(font
+					(size 1.27 1.27)
+				)
+				(hide yes)
+			)
+		)
+		(property "Datasheet" ""
+			(at 226.06 81.28 0)
+			(effects
+				(font
+					(size 1.27 1.27)
+				)
+				(hide yes)
+			)
+		)
+		(property "Description" ""
+			(at 226.06 81.28 0)
+			(effects
+				(font
+					(size 1.27 1.27)
+				)
+				(hide yes)
+			)
+		)
+		(pin "1"
+		)
+		(instances
+			(project ""
+				(path "/d3cb7130-decc-418b-958e-e5d84a8d867f/af07603d-259f-481d-be2c-d925e27835a3"
+					(reference "ANT1")
+					(unit 1)
+				)

Commit message: EG-49 Tests points added.
Parts:
- added TP14: RF_VDD, TestPoint:TestPoint_Pad_D1.0mm, symbol Connector:TestPoint
Connections:
- net RF_VDD: now also TP14.1
Changed lines of the file:
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@@
+	(wire
+		(pts
+			(xy 55.88 39.37) (xy 55.88 45.72)
+		)
+		(stroke
+			(width 0)
+			(type default)
+		)
+	)
 	(wire
 		(pts
@@
 					(unit 1)
 				)
+			)
+		)
+	)
+	(symbol
+		(lib_id "Connector:TestPoint")
+		(at 55.88 45.72 180)
+		(unit 1)
+		(exclude_from_sim no)
+		(in_bom yes)
+		(on_board yes)
+		(dnp no)
+		(fields_autoplaced yes)
+		(property "Reference" "TP14"
+			(at 58.42 47.7519 0)
+			(effects
+				(font
+					(size 1.27 1.27)
+				)
+				(justify right)
+			)
+		)
+		(property "Value" "RF_VDD"
+			(at 58.42 50.2919 0)
+			(effects
+				(font
+					(size 1.27 1.27)
+				)
+				(justify right)
+			)
+		)
+		(property "Footprint" "TestPoint:TestPoint_Pad_D1.0mm"
+			(at 50.8 45.72 0)
+			(effects
+				(font
+					(size 1.27 1.27)
+				)
+				(hide yes)
+			)
+		)
+		(property "Datasheet" "~"
+			(at 50.8 45.72 0)
+			(effects
+				(font
+					(size 1.27 1.27)
+				)
+				(hide yes)
+			)
+		)
+		(property "Description" "test point"
+			(at 55.88 45.72 0)
+			(effects
+				(font
+					(size 1.27 1.27)
+				)
+				(hide yes)
+			)
+		)
+		(pin "1"
+		)
+		(instances
+			(project "sensor_rev1"
+				(path "/d3cb7130-decc-418b-958e-e5d84a8d867f/af07603d-259f-481d-be2c-d925e27835a3"
+					(reference "TP14")
+					(unit 1)
+				)

Commit message: EG-49 ERC with no errors.
Other:
- moved on the sheet: C6, C9, TP14

Commit message: EG-49 No ERC warnings.
Parts:
- FB1: Manufacturer (none) -> Murata Electronics; Manufacturer Part Number (none) -> BLM18KG601SN1D; Supplier Link (none) -> https://www.mouser.co.uk/ProductDetail/Murata-Electronics/B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
- IC2: Manufacturer (none) -> Texas Instruments; Manufacturer Part Number (none) -> CC1101RGPR; Supplier Link (none) -> https://www.mouser.co.uk/ProductDetail/Texas-Instruments/CC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
- Y1: Manufacturer (none) -> NDK; Manufacturer Part Number (none) -> NX3225GA-26.000M-STD-CRG-2; Supplier Link (none) -> https://www.mouser.co.uk/ProductDetail/NDK/NX3225GA-26.000M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
Changed lines of the file:
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@@
+			)
+		)
+		(property "Supplier Link" "https://www.mouser.co.uk/ProductDetail/Texas-Instruments/CC1101RGPR?qs=OHhYoCux73lreNWI41kZ9Q%3D%3D"
+			(at 114.3 659.69 0)
+			(effects
+				(font
+					(size 1.27 1.27)
+				)
+				(justify left top)
+				(hide yes)
+			)
+		)
+		(property "Manufacturer" "Texas Instruments"
+			(at 114.3 759.69 0)
+			(effects
+				(font
+					(size 1.27 1.27)
+				)
+				(justify left top)
+				(hide yes)
+			)
+		)
+		(property "Manufacturer Part Number" "CC1101RGPR"
+			(at 114.3 859.69 0)
+			(effects
+				(font
+					(size 1.27 1.27)
+				)
+				(justify left top)
+				(hide yes)
 			)
 		)
@@
 			)
 		)
+		(property "Supplier Link" "https://www.mouser.co.uk/ProductDetail/Murata-Electronics/BLM18KG601SN1D?qs=rvfpa0%252BU10NPWIt745bDHg%3D%3D"
+			(at 26.67 631.75 0)
+			(effects
+				(font
+					(size 1.27 1.27)
+				)
+				(justify left top)
+				(hide yes)
+			)
+		)
+		(property "Manufacturer" "Murata Electronics"
+			(at 26.67 731.75 0)
+			(effects
+				(font
+					(size 1.27 1.27)
+				)
+				(justify left top)
+				(hide yes)
+			)
+		)
+		(property "Manufacturer Part Number" "BLM18KG601SN1D"
+			(at 26.67 831.75 0)
+			(effects
+				(font
+					(size 1.27 1.27)
+				)
+				(justify left top)
+				(hide yes)
+			)
+		)
 		(pin "2"
 		)
@@
 			(at 118.11 923.19 0)
 			(effects
+				(font
+					(size 1.27 1.27)
+				)
+				(justify left top)
+				(hide yes)
+			)
+		)
+		(property "Supplier Link" "https://www.mouser.co.uk/ProductDetail/NDK/NX3225GA-26.000M-STD-CRG-2?qs=w%2Fv1CP2dgqrNyFiUoufKQw%3D%3D"
+			(at 118.11 723.19 0)
+			(effects
+				(font
+					(size 1.27 1.27)
+				)
+				(justify left top)
+				(hide yes)
+			)
+		)
+		(property "Manufacturer" "NDK"
+			(at 118.11 823.19 0)
+			(effects
+				(font
+					(size 1.27 1.27)
+				)
+				(justify left top)
+				(hide yes)
+			)
+		)
+		(property "Manufacturer Part Number" "NX3225GA-26.000M-STD-CRG-2"
+			(at 118.11 923.19 0)
+			(effects
