File: hardware/sensor/rev1/rf_rev1.kicad_sch (KiCad schematic)
At the start: 27 parts, among them IC2 CC1101RGPR, Y1 NX3225GA-26.000M-STD-CRG-2

Commit message: EG-50 Components ready to be connected.
Connections:
- net GND: no longer Y1.2 (NC/GND_1), Y1.4 (NC/GND_2)
- no-connect marks 1 -> 3
Changed lines of the file:
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@@
 	)
 	(no_connect
+		(at 78.74 128.27)
+	)
+	(no_connect
 		(at 80.01 80.01)
 	)
+	(no_connect
+		(at 121.92 130.81)
+	)
 	(wire
 		(pts
@@
 	(wire
 		(pts
-			(xy 125.73 130.81) (xy 125.73 148.59)
-		)
-		(stroke
-			(width 0)
-			(type default)
-		)
-	)
-	(wire
-		(pts
 			(xy 111.76 41.91) (xy 111.76 46.99)
 		)
@@
 	(wire
 		(pts
-			(xy 121.92 130.81) (xy 125.73 130.81)
-		)
-		(stroke
-			(width 0)
-			(type default)
-		)
-	)
-	(wire
-		(pts
 			(xy 139.7 72.39) (xy 121.92 72.39)
 		)
@@
 	(wire
 		(pts
-			(xy 74.93 128.27) (xy 78.74 128.27)
-		)
-		(stroke
-			(width 0)
-			(type default)
-		)
-	)
-	(wire
-		(pts
 			(xy 163.83 106.68) (xy 163.83 110.49)
 		)
@@
 	(wire
 		(pts
-			(xy 74.93 148.59) (xy 74.93 128.27)
-		)
-		(stroke
-			(width 0)
-			(type default)
-		)
-	)
-	(wire
-		(pts
 			(xy 118.11 85.09) (xy 121.92 85.09)
 		)
@@
 	)
 	(symbol
-		(lib_id "power:GND")
-		(at 125.73 148.59 0)
-		(unit 1)
-		(exclude_from_sim no)
-		(in_bom yes)
-		(on_board yes)
-		(dnp no)
-		(fields_autoplaced yes)
-		(property "Reference" "#PWR046"
-			(at 125.73 154.94 0)
-			(effects
-				(font
-					(size 1.27 1.27)
-				)
-				(hide yes)
-			)
-		)
-		(property "Value" "GND"
-			(at 125.73 153.67 0)
-			(effects
-				(font
-					(size 1.27 1.27)
-				)
-			)
-		)
-		(property "Footprint" ""
-			(at 125.73 148.59 0)
-			(effects
-				(font
-					(size 1.27 1.27)
-				)
-				(hide yes)
-			)
-		)
-		(property "Datasheet" ""
-			(at 125.73 148.59 0)
-			(effects
-				(font
-					(size 1.27 1.27)
-				)
-				(hide yes)
-			)
-		)
-		(property "Description" "Power symbol creates a global label with name \"GND\" , ground"
-			(at 125.73 148.59 0)
-			(effects
-				(font
-					(size 1.27 1.27)
-				)
-				(hide yes)
-			)
-		)
-		(pin "1"
-		)
-		(instances
-			(project "rf_rev1"
-				(path "/50a12035-955f-49d8-a6b8-24fcd6d450af"
-					(reference "#PWR?")
-					(unit 1)
-				)
-			)
-			(project "sensor_rev1"
-				(path "/d3cb7130-decc-418b-958e-e5d84a8d867f/af07603d-259f-481d-be2c-d925e27835a3"
-					(reference "#PWR046")
-					(unit 1)
-				)
-			)
-		)
-	)
-	(symbol
 		(lib_id "Device:C")
 		(at 68.58 92.71 0)
@@
 					(unit 1)
 				)
-			)
-		)
-	)
-	(symbol
-		(lib_id "power:GND")
-		(at 74.93 148.59 0)
-		(unit 1)
-		(exclude_from_sim no)
-		(in_bom yes)
-		(on_board yes)
-		(dnp no)
-		(fields_autoplaced yes)
-		(property "Reference" "#PWR047"
-			(at 74.93 154.94 0)
-			(effects
-				(font
-					(size 1.27 1.27)
-				)
-				(hide yes)
-			)
-		)
-		(property "Value" "GND"
-			(at 74.93 153.67 0)
-			(effects
-				(font
-					(size 1.27 1.27)
-				)
-			)
-		)
-		(property "Footprint" ""
-			(at 74.93 148.59 0)
-			(effects
-				(font
-					(size 1.27 1.27)
-				)
-				(hide yes)
-			)
-		)
-		(property "Datasheet" ""
-			(at 74.93 148.59 0)
-			(effects
-				(font
-					(size 1.27 1.27)
-				)
-				(hide yes)
-			)
-		)
-		(property "Description" "Power symbol creates a global label with name \"GND\" , ground"
-			(at 74.93 148.59 0)
-			(effects
-				(font
-					(size 1.27 1.27)
-				)
-				(hide yes)
-			)
-		)
-		(pin "1"
-		)
-		(instances
-			(project "rf_rev1"
-				(path "/50a12035-955f-49d8-a6b8-24fcd6d450af"
-					(reference "#PWR?")
-					(unit 1)
-				)
-			)
-			(project "sensor_rev1"
-				(path "/d3cb7130-decc-418b-958e-e5d84a8d867f/af07603d-259f-481d-be2c-d925e27835a3"
-					(reference "#PWR047")
-					(unit 1)
-				)

Commit message: EG-50 Only warings on CR2032 battery holder.
Parts:
- FB1: Manufacturer_Name Murata Electronics -> (none); Manufacturer_Part_Number BLM18KG601SN1D -> (none); Mouser Price/Stock https://www.mouser.co.uk/ProductDetail/Murata-Electronics/B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 -> (none)
- IC2: Manufacturer_Name Texas Instruments -> (none); Manufacturer_Part_Number CC1101RGPR -> (none); Mouser Price/Stock https://www.mouser.co.uk/ProductDetail/Texas-Instruments/CC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 -> (none)
- Y1: Manufacturer_Name NDK -> (none); Manufacturer_Part_Number NX3225GA-26.000M-STD-CRG-2 -> (none); Mouser Price/Stock https://www.mouser.co.uk/en/ProductDetail/NDK/STDCRG2-26M?q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 -> (none)
Connections:
- net RF_VDD: now also FB1.1; no longer FB1.2
- net VDD: now also FB1.2; no longer FB1.1

Commit message: EG-50 PCB Finalized.
Parts:
- renumbered TP14 to RFVDD1
Changed lines of the file:
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@@
 		(dnp no)
 		(fields_autoplaced yes)
-		(property "Reference" "TP14"
+		(property "Reference" "RFVDD1"
 			(at 54.61 47.7519 0)
 			(effects
@@
 			(project "sensor_rev1"
 				(path "/d3cb7130-decc-418b-958e-e5d84a8d867f/af07603d-259f-481d-be2c-d925e27835a3"
-					(reference "TP14")
+					(reference "RFVDD1")
 					(unit 1)
 				)

Commit message: EG-50 Bill of Materials.
Parts:
- FB1: Manufacturer Murata Electronics -> (none); Manufacturer_Name (none) -> Murata Electronics; Mouser Price/Stock (none) -> https://www.mouser.co.uk/ProductDetail/Murata-Electronics/B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; Supplier Link https://www.mouser.co.uk/ProductDetail/Murata-Electronics/B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 -> (none)
- IC2: Manufacturer Texas Instruments -> (none); Manufacturer_Name (none) -> Texas Instruments; Mouser Price/Stock (none) -> https://www.mouser.co.uk/ProductDetail/Texas-Instruments/CC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; Supplier Link https://www.mouser.co.uk/ProductDetail/Texas-Instruments/CC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 -> (none)
- Y1: Manufacturer NDK -> (none); Manufacturer_Name (none) -> NDK; Mouser Price/Stock (none) -> https://www.mouser.co.uk/ProductDetail/NDK/NX3225GA-26.000M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; Supplier Link https://www.mouser.co.uk/ProductDetail/NDK/NX3225GA-26.000M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 -> (none)

Commit message: EG-70 XTAL replaced according with JLCPCB constraints and capacitors adjusted accordingly.
Parts:
- C101: value 12pF -> 15pF; Manufacturer_Name Murata Electronics -> Vishay; Manufacturer_Part_Number GRM1555C1H120FA1D -> VJ0402D150FXCAJ; Mouser Part Number 81-GRM1555C1H120FA1D -> 77-VJ0402D150FXCAJ
- C81: value 12pF -> 15pF; Manufacturer_Name Murata Electronics -> Vishay; Manufacturer_Part_Number GRM1555C1H120FA1D -> VJ0402D150FXCAJ; Mouser Part Number 81-GRM1555C1H120FA1D -> 77-VJ0402D150FXCAJ; Mouser Price/Stock https://pt.mouser.com/ProductDetail/Murata-Electronics/GRM1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 -> https://pt.mouser.com/en/ProductDetail/Vishay-Vitramon/VJ04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
- Y1: value NX3225GA-26.000M-STD-CRG-2 -> CG01972-26M; Manufacturer Part Number NX3225GA-26.000M-STD-CRG-2 -> CG01972-26M; Mouser Part Number 344-NX3225GA26MSTRG2 -> 344-NX3225GA26MHZTI; Mouser Price/Stock https://www.mouser.co.uk/ProductDetail/NDK/NX3225GA-26.000M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 -> https://pt.mouser.com/en/ProductDetail/NDK/CG01972-26M?qs=T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
Changed lines of the file:
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@@
 			)
 		)
-		(property "Value" "12pF"
+		(property "Value" "15pF"
 			(at 137.16 142.2399 0)
 			(effects
@@
 			)
 		)
-		(property "Mouser Part Number" "81-GRM1555C1H120FA1D"
+		(property "Mouser Part Number" "77-VJ0402D150FXCAJ"
 			(at 133.35 140.97 0)
 			(effects
@@
 			)
 		)
-		(property "Manufacturer_Name" "Murata Electronics"
+		(property "Manufacturer_Name" "Vishay"
 			(at 133.35 140.97 0)
 			(effects
@@
 			)
 		)
-		(property "Manufacturer_Part_Number" "GRM1555C1H120FA1D"
+		(property "Manufacturer_Part_Number" "VJ0402D150FXCAJ"
 			(at 133.35 140.97 0)
 			(effects
@@
 			)
 		)
-		(property "Value" "NX3225GA-26.000M-STD-CRG-2"
+		(property "Value" "CG01972-26M"
 			(at 100.33 123.19 0)
 			(effects
@@
 			)
 		)
-		(property "Mouser Part Number" "344-NX3225GA26MSTRG2"
+		(property "Mouser Part Number" "344-NX3225GA26MHZTI"
 			(at 118.11 623.19 0)
 			(effects
@@
 			)
 		)
-		(property "Mouser Price/Stock" "https://www.mouser.co.uk/ProductDetail/NDK/NX3225GA-26.000M-STD-CRG-2?qs=w%2Fv1CP2dgqrNyFiUoufKQw%3D%3D"
+		(property "Mouser Price/Stock" "https://pt.mouser.com/en/ProductDetail/NDK/CG01972-26M?qs=Tc%252BHE9vUsntpTnxiVVqD7w%3D%3D"
 			(at 118.11 723.19 0)
 			(effects
@@
 			)
 		)
-		(property "Manufacturer Part Number" "NX3225GA-26.000M-STD-CRG-2"
+		(property "Manufacturer Part Number" "CG01972-26M"
 			(at 118.11 923.19 0)
 			(effects
@@
 			)
 		)
-		(property "Value" "12pF"
+		(property "Value" "15pF"
 			(at 66.04 142.2399 0)
 			(effects
@@
 			)
 		)
-		(property "Mouser Part Number" "81-GRM1555C1H120FA1D"
+		(property "Mouser Part Number" "77-VJ0402D150FXCAJ"
 			(at 69.85 140.97 0)
 			(effects
@@
 			)
 		)
-		(property "Mouser Price/Stock" "https://pt.mouser.com/ProductDetail/Murata-Electronics/GRM1555C1H120FA01D?qs=ouTquLLW2S4GiX6b03cbUg%3D%3D"
+		(property "Mouser Price/Stock" "https://pt.mouser.com/en/ProductDetail/Vishay-Vitramon/VJ0402D150FXCAJ?qs=iYZfuFMDqcZeWrff4BZNMQ%3D%3D"
 			(at 69.85 140.97 0)
 			(effects
@@
 			)
 		)
-		(property "Manufacturer_Name" "Murata Electronics"
+		(property "Manufacturer_Name" "Vishay"
 			(at 69.85 140.97 0)
 			(effects
@@
 			)
 		)
-		(property "Manufacturer_Part_Number" "GRM1555C1H120FA1D"
+		(property "Manufacturer_Part_Number" "VJ0402D150FXCAJ"
 			(at 69.85 140.97 0)
 			(effects

Commit message: EG-70 Adaptions on XTAL name.
Parts:
- Y1: value CG01972-26M -> NX3225GA-26MHZ-TI; Manufacturer Part Number CG01972-26M -> NX3225GA-26MHZ-TI
Changed lines of the file:
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@@
 			)
 		)
-		(property "Value" "CG01972-26M"
+		(property "Value" "NX3225GA-26MHZ-TI"
 			(at 100.33 123.19 0)
 			(effects
@@
 			)
 		)
-		(property "Manufacturer Part Number" "CG01972-26M"
+		(property "Manufacturer Part Number" "NX3225GA-26MHZ-TI"
 			(at 118.11 923.19 0)
 			(effects

Commit message: Connected the XTAL NC/GND pins to GND. Added a via for decouple capacitors of CC1101.
Parts:
- ANT1: value ~ -> (none)
Connections:
- net GND: now also Y1.2 (NC/GND_1), Y1.4 (NC/GND_2)
- no-connect marks 3 -> 1

Commit message: Final adjustments to PCB and schematic after review session.
Connections:
- net GND: no longer Y1.2 (NC/GND_1), Y1.4 (NC/GND_2)
- no-connect marks 1 -> 3
Changed lines of the file:
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@@
 	)
 	(no_connect
+		(at 121.92 130.81)
+	)
+	(no_connect
 		(at 80.01 80.01)
 	)
+	(no_connect
+		(at 78.74 128.27)
+	)
 	(wire
 		(pts
@@
 	(wire
 		(pts
-			(xy 127 135.89) (xy 127 130.81)
-		)
-		(stroke
-			(width 0)
-			(type default)
-		)
-	)
-	(wire
-		(pts
 			(xy 179.07 86.36) (xy 181.61 86.36)
 		)
@@
 	(wire
 		(pts
-			(xy 127 130.81) (xy 121.92 130.81)
-		)
-		(stroke
-			(width 0)
-			(type default)
-		)
-	)
-	(wire
-		(pts
 			(xy 76.2 82.55) (xy 76.2 54.61)
 		)
@@
 	(wire
 		(pts
-			(xy 76.2 128.27) (xy 78.74 128.27)
-		)
-		(stroke
-			(width 0)
-			(type default)
-		)
-	)
-	(wire
-		(pts
 			(xy 165.1 76.2) (xy 171.45 76.2)
 		)
@@
 	(wire
 		(pts
-			(xy 76.2 135.89) (xy 76.2 128.27)
-		)
-		(stroke
-			(width 0)
-			(type default)
-		)
-	)
-	(wire
-		(pts
 			(xy 181.61 81.28) (xy 182.88 81.28)
 		)
@@
 	(symbol
 		(lib_id "power:GND")
-		(at 127 135.89 0)
-		(unit 1)
-		(body_style 1)
-		(exclude_from_sim no)
-		(in_bom yes)
-		(on_board yes)
-		(in_pos_files yes)
-		(dnp no)
-		(fields_autoplaced yes)
-		(property "Reference" "#PWR044"
-			(at 127 142.24 0)
-			(hide yes)
-			(show_name no)
-			(do_not_autoplace no)
-			(effects
-				(font
-					(size 1.27 1.27)
-				)
-			)
-		)
-		(property "Value" "GND"
-			(at 127 140.97 0)
-			(show_name no)
-			(do_not_autoplace no)
-			(effects
-				(font
-					(size 1.27 1.27)
-				)
-			)
-		)
-		(property "Footprint" ""
-			(at 127 135.89 0)
-			(hide yes)
-			(show_name no)
-			(do_not_autoplace no)
-			(effects
-				(font
-					(size 1.27 1.27)
-				)
-			)
-		)
-		(property "Datasheet" ""
-			(at 127 135.89 0)
-			(hide yes)
-			(show_name no)
-			(do_not_autoplace no)
-			(effects
-				(font
-					(size 1.27 1.27)
-				)
-			)
-		)
-		(property "Description" "Power symbol creates a global label with name \"GND\" , ground"
-			(at 127 135.89 0)
-			(hide yes)
-			(show_name no)
-			(do_not_autoplace no)
-			(effects
-				(font
-					(size 1.27 1.27)
-				)
-			)
-		)
-		(pin "1"
-		)
-		(instances
-			(project "sensor_rev1"
-				(path "/d3cb7130-decc-418b-958e-e5d84a8d867f/af07603d-259f-481d-be2c-d925e27835a3"
-					(reference "#PWR044")
-					(unit 1)
-				)
-			)
-		)
-	)
-	(symbol
-		(lib_id "power:GND")
 		(at 68.58 100.33 0)
 		(unit 1)
@@
 					(unit 1)
 				)
-			)
-		)
-	)
-	(symbol
-		(lib_id "power:GND")
-		(at 76.2 135.89 0)
-		(unit 1)
-		(body_style 1)
-		(exclude_from_sim no)
-		(in_bom yes)
-		(on_board yes)
-		(in_pos_files yes)
-		(dnp no)
-		(fields_autoplaced yes)
-		(property "Reference" "#PWR045"
-			(at 76.2 142.24 0)
-			(hide yes)
-			(show_name no)
-			(do_not_autoplace no)
-			(effects
-				(font
-					(size 1.27 1.27)
-				)
-			)
-		)
-		(property "Value" "GND"
-			(at 76.2 140.97 0)
-			(show_name no)
-			(do_not_autoplace no)
-			(effects
-				(font
-					(size 1.27 1.27)
-				)
-			)
-		)
-		(property "Footprint" ""
-			(at 76.2 135.89 0)
-			(hide yes)
-			(show_name no)
-			(do_not_autoplace no)
-			(effects
-				(font
-					(size 1.27 1.27)
-				)
-			)
-		)
-		(property "Datasheet" ""
-			(at 76.2 135.89 0)
-			(hide yes)
-			(show_name no)
-			(do_not_autoplace no)
-			(effects
-				(font
-					(size 1.27 1.27)
-				)
-			)
-		)
-		(property "Description" "Power symbol creates a global label with name \"GND\" , ground"
-			(at 76.2 135.89 0)
-			(hide yes)
-			(show_name no)
-			(do_not_autoplace no)
-			(effects
-				(font
-					(size 1.27 1.27)
-				)
-			)
-		)
-		(pin "1"
-		)
-		(instances
-			(project "sensor_rev1"
-				(path "/d3cb7130-decc-418b-958e-e5d84a8d867f/af07603d-259f-481d-be2c-d925e27835a3"
-					(reference "#PWR045")
-					(unit 1)
-				)
