File: hardware/gateway/rev2/buzzer_rev2.kicad_sch (KiCad schematic)
At the start: 16 parts, among them IC3 LT1615ES5-1#TRMPBF, IC4 MIC4427YM

Commit message: EG-59 Adapted the buzzer driver.
Parts:
- removed C26: 22uF, 6.3V, Capacitor_SMD:C_1206_3216Metric, symbol Device:C
- removed C27: 4.7pF, Capacitor_SMD:C_0402_1005Metric, symbol Device:C
- removed C28, C29: 4.7uF, 25V, Capacitor_SMD:C_0805_2012Metric, symbol Device:C
- removed C30: 100nF, Capacitor_SMD:C_0402_1005Metric, symbol Device:C
- removed D1: MBR0520LT3G, MyParts:SOD3716X135N, symbol MBR0520LT3G:MBR0520LT3G
- removed IC3: LT1615ES5-1#TRMPBF, MyParts:SOT95P280X100-5N, symbol LT1615ES5-1#TRMPBF:LT1615ES5-1#TRMPBF
- removed IC4: MIC4427YM, MyParts:SOIC127P599X173-8N, symbol MIC4427YM:MIC4427YM
- removed L5: CD43NP-100MC, MyParts:CD43NP100MC, symbol CD43NP-100MC:CD43NP-100MC
- removed LS1: PKMCS1818E20A0-R1, MyParts:PKMCS1818E20A0R1, symbol PKMCS1818E20A0-R1:PKMCS1818E20A0-R1
- removed R15: 100K, Resistor_SMD:R_0603_1608Metric, symbol Device:R_US
- removed R16: 130K, Resistor_SMD:R_0402_1005Metric, symbol Device:R_US
- removed R17: 1.15M, Resistor_SMD:R_0402_1005Metric, symbol Device:R_US
- removed R18, R19: 33R, Resistor_SMD:R_0603_1608Metric, symbol Device:R_US
- removed R20: 1M, Resistor_SMD:R_0603_1608Metric, symbol Device:R_US
Connections:
- no-connect marks 2 -> 0
