File: hardware/gateway/rev2/gateway_rev2.kicad_sch (KiCad schematic)
At the start: 7 parts

Commit message: EG-59 Schematic with the needed components, plus PCB.
Other:
- removed sheet Buzzer
- sheet MCU ports: added none; removed BZR_EN, BZR_N, BZR_P
Changed lines of the file:
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@@
 	(wire
 		(pts
-			(xy 86.36 27.94) (xy 95.25 27.94)
+			(xy 49.53 27.94) (xy 58.42 27.94)
 		)
 		(stroke
@@
 	(wire
 		(pts
-			(xy 50.8 29.21) (xy 60.96 29.21)
+			(xy 49.53 22.86) (xy 58.42 22.86)
 		)
 		(stroke
@@
 	(wire
 		(pts
-			(xy 86.36 22.86) (xy 95.25 22.86)
+			(xy 49.53 33.02) (xy 58.42 33.02)
 		)
 		(stroke
@@
 	(wire
 		(pts
-			(xy 86.36 33.02) (xy 95.25 33.02)
+			(xy 49.53 30.48) (xy 58.42 30.48)
 		)
 		(stroke
@@
 	(wire
 		(pts
-			(xy 86.36 30.48) (xy 95.25 30.48)
-		)
-		(stroke
-			(width 0)
-			(type default)
-		)
-	)
-	(wire
-		(pts
-			(xy 50.8 22.86) (xy 60.96 22.86)
-		)
-		(stroke
-			(width 0)
-			(type default)
-		)
-	)
-	(wire
-		(pts
-			(xy 50.8 26.67) (xy 60.96 26.67)
-		)
-		(stroke
-			(width 0)
-			(type default)
-		)
-	)
-	(wire
-		(pts
-			(xy 86.36 25.4) (xy 95.25 25.4)
+			(xy 49.53 25.4) (xy 58.42 25.4)
 		)
 		(stroke
@@
 	)
 	(sheet
-		(at 95.25 19.05)
+		(at 58.42 19.05)
 		(size 25.4 17.78)
 		(exclude_from_sim no)
@@
 		)
 		(property "Sheetname" "RF"
-			(at 95.25 18.3384 0)
+			(at 58.42 18.3384 0)
 			(show_name no)
 			(do_not_autoplace no)
@@
 		)
 		(property "Sheetfile" "rf_rev2.kicad_sch"
-			(at 95.25 37.4146 0)
+			(at 58.42 37.4146 0)
 			(show_name no)
 			(do_not_autoplace no)
@@
 		)
 		(pin "CS" input
-			(at 95.25 30.48 180)
+			(at 58.42 30.48 180)
 			(effects
 				(font
@@
 		)
 		(pin "SCLK" input
-			(at 95.25 22.86 180)
+			(at 58.42 22.86 180)
 			(effects
 				(font
@@
 		)
 		(pin "SDI" input
-			(at 95.25 25.4 180)
+			(at 58.42 25.4 180)
 			(effects
 				(font
@@
 		)
 		(pin "SDO" input
-			(at 95.25 27.94 180)
+			(at 58.42 27.94 180)
 			(effects
 				(font
@@
 		)
 		(pin "IRQ" input
-			(at 95.25 33.02 180)
+			(at 58.42 33.02 180)
 			(effects
 				(font
@@
 	)
 	(sheet
-		(at 60.96 19.05)
+		(at 24.13 19.05)
 		(size 25.4 17.78)
 		(exclude_from_sim no)
@@
 		)
 		(property "Sheetname" "MCU"
-			(at 60.96 18.3384 0)
+			(at 24.13 18.3384 0)
 			(show_name no)
 			(do_not_autoplace no)
@@
 		)
 		(property "Sheetfile" "mcu_rev2.kicad_sch"
-			(at 60.96 37.4146 0)
+			(at 24.13 37.4146 0)
 			(show_name no)
 			(do_not_autoplace no)
@@
 			)
 		)
-		(pin "BZR_EN" input
-			(at 60.96 22.86 180)
-			(effects
-				(font
-					(size 1.27 1.27)
-				)
-				(justify left)
-			)
-		)
-		(pin "BZR_N" input
-			(at 60.96 29.21 180)
-			(effects
-				(font
-					(size 1.27 1.27)
-				)
-				(justify left)
-			)
-		)
-		(pin "BZR_P" input
-			(at 60.96 26.67 180)
-			(effects
-				(font
-					(size 1.27 1.27)
-				)
-				(justify left)
-			)
-		)
 		(pin "CS" input
-			(at 86.36 30.48 0)
+			(at 49.53 30.48 0)
 			(effects
 				(font
@@
 		)
 		(pin "SCLK" input
-			(at 86.36 22.86 0)
+			(at 49.53 22.86 0)
 			(effects
 				(font
@@
 		)
 		(pin "SDI" input
-			(at 86.36 25.4 0)
+			(at 49.53 25.4 0)
 			(effects
 				(font
@@
 		)
 		(pin "SDO" input
-			(at 86.36 27.94 0)
+			(at 49.53 27.94 0)
 			(effects
 				(font
@@
 		)
 		(pin "IRQ" input
-			(at 86.36 33.02 0)
+			(at 49.53 33.02 0)
 			(effects
 				(font
@@
 				)
 			)
-		)
-	)
-	(sheet
-		(at 24.13 19.05)
-		(size 26.67 17.78)
-		(exclude_from_sim no)
-		(in_bom yes)
-		(on_board yes)
-		(dnp no)
-		(fields_autoplaced yes)
-		(stroke
-			(width 0.1524)
-			(type solid)
-		)
-		(fill
-			(color 0 0 0 0)
-		)
-		(property "Sheetname" "Buzzer"
-			(at 24.13 18.3384 0)
-			(show_name no)
-			(do_not_autoplace no)
-			(effects
-				(font
-					(size 1.27 1.27)
-				)
-				(justify left bottom)
-			)
-		)
-		(property "Sheetfile" "buzzer_rev2.kicad_sch"
-			(at 24.13 37.4146 0)
-			(show_name no)
-			(do_not_autoplace no)
-			(effects
-				(font
-					(size 1.27 1.27)
-				)
-				(justify left top)
-			)
-		)
-		(pin "BZR_EN" input
-			(at 50.8 22.86 0)
-			(effects
-				(font
-					(size 1.27 1.27)
-				)
-				(justify right)
-			)
-		)
-		(pin "BZR_N" input
-			(at 50.8 29.21 0)
-			(effects
-				(font
-					(size 1.27 1.27)
-				)
-				(justify right)
-			)
-		)
-		(pin "BZR_P" input
-			(at 50.8 26.67 0)
-			(effects
-				(font
-					(size 1.27 1.27)
-				)
-				(justify right)
-			)
-		)
-		(instances
-			(project "gateway_rev2"
-				(path "/d3cb7130-decc-418b-958e-e5d84a8d867f"
-					(page "4")
-				)
-			)
