File: hardware/gateway/rev2/mcu_rev2.kicad_sch (KiCad schematic)
At the start: 34 parts, among them IC1 STM8L151K4T6, IC5 MB85RC64TAPNF-G-BDERE1, J1 22-28-4044, J2 M20-9770342, U1 IRM-01-3.3

Commit message: EG-59 Components supplier fixed.
Parts:
- C1: Manufacturer Murata -> (none); Manufacturer Part Number GXT155R71C103KE01D -> (none); Manufacturer_Name (none) -> Taiyo Yuden; Manufacturer_Part_Number (none) -> MSAST105SB7103KFNA01; Mouser Part Number 81-GXT155R71C103KE1D -> 963-MSAST105SB7103KF; Mouser Price/Stock (none) -> https://pt.mouser.com/en/ProductDetail/TAIYO-YUDEN/MSAST105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; Supplier Link https://pt.mouser.com/ProductDetail/Murata-Electronics/GXT1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 -> https://pt.mouser.com/en/ProductDetail/TAIYO-YUDEN/MSAST105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
- C2: Manufacturer Yageo -> (none); Manufacturer Part Number CC603KRX5R6BB105 -> (none); Manufacturer_Name (none) -> Kyocera Avx; Manufacturer_Part_Number (none) -> KGM05AV50J105ZH; Mouser Part Number 603-CC603KRX5R6BB105 -> 581-KGM05AV50J105ZH; Mouser Price/Stock (none) -> https://pt.mouser.com/en/ProductDetail/KYOCERA-AVX/KGM05AV5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; Supplier Link https://pt.mouser.com/ProductDetail/YAGEO/CC0603KRX5R6BB105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 -> https://pt.mouser.com/en/ProductDetail/KYOCERA-AVX/KGM05AV5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
- C3: Manufacturer Taiyo Yuden -> (none); Manufacturer Part Number MAJCH168BB7104KT -> (none); Manufacturer_Name (none) -> Yageo; Manufacturer_Part_Number (none) -> CC0402KRX7R7BB104; Mouser Part Number 963-MAJCH168BB7104KT -> 603-CC402KRX7R7BB104; Mouser Price/Stock (none) -> https://pt.mouser.com/en/ProductDetail/YAGEO/CC0402KRX7R7BB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; Supplier Link https://pt.mouser.com/ProductDetail/TAIYO-YUDEN/MAJCH168BB7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 -> https://pt.mouser.com/en/ProductDetail/YAGEO/CC0402KRX7R7BB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
- C4: Manufacturer Murata -> (none); Manufacturer Part Number GXT155R60J105KE01D -> (none); Manufacturer_Name (none) -> Kyocera Avx; Manufacturer_Part_Number (none) -> KGM05AV50J105ZH; Mouser Part Number 81-GXT155R60J105KE1D -> 581-KGM05AV50J105ZH; Mouser Price/Stock (none) -> https://pt.mouser.com/en/ProductDetail/KYOCERA-AVX/KGM05AV5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; Supplier Link https://pt.mouser.com/ProductDetail/Murata-Electronics/GXT1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 -> https://pt.mouser.com/en/ProductDetail/KYOCERA-AVX/KGM05AV5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
- C50: Manufacturer Yageo -> (none); Manufacturer Part Number CC0402KRX7R7BB104 -> (none); Manufacturer_Name (none) -> Yageo; Manufacturer_Part_Number (none) -> CC0402KRX7R7BB104; Mouser Price/Stock (none) -> https://pt.mouser.com/en/ProductDetail/YAGEO/CC0402KRX7R7BB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; Supplier Link https://pt.mouser.com/ProductDetail/YAGEO/CC0402KRX7R7BB104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 -> https://pt.mouser.com/en/ProductDetail/YAGEO/CC0402KRX7R7BB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
- IC1: Manufacturer STMicroelectronics -> (none); Manufacturer Part Number STM8L151K4T6 -> (none); Manufacturer_Name (none) -> STMicroelectronics; Manufacturer_Part_Number (none) -> STM8L151K4T6; Mouser Price/Stock (none) -> https://pt.mouser.com/en/ProductDetail/STMicroelectronics/S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; Supplier Link https://www.mouser.co.uk/ProductDetail/STMicroelectronics/S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 -> https://pt.mouser.com/en/ProductDetail/STMicroelectronics/S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
- IC5: Manufacturer_Name (none) -> RAMXEED; Manufacturer_Part_Number (none) -> MB85RC64TAPNF-G-BDERE1; Mouser Price/Stock (none) -> https://pt.mouser.com/en/ProductDetail/RAMXEED/MB85RC64TAPN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
- J1: Mouser Price/Stock https://www.mouser.com/Search/Refine.aspx?Keyword=538-22-28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 -> https://pt.mouser.com/en/ProductDetail/Molex/22-28-4044?qs=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
- LED1: Manufacturer Part Number WP710A10LVBC/D -> (none); Manufacturer_Name (none) -> Kingbright; Manufacturer_Part_Number (none) -> WP710A10LVBC/D; Mouser Price/Stock (none) -> https://www.mouser.co.uk/ProductDetail/Kingbright/WP710A10L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
- LED2: Manufacturer Vishay -> (none); Manufacturer Part Number TLHY4400-AS12Z -> (none); Manufacturer_Name (none) -> Vishay; Manufacturer_Part_Number (none) -> TLHY4400-AS12Z; Mouser Price/Stock (none) -> https://pt.mouser.com/en/ProductDetail/Vishay-Semiconductor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
- LED3: Manufacturer Vishay -> (none); Manufacturer Part Number TLHR4400-AS12Z -> (none); Manufacturer_Name (none) -> Vishay; Manufacturer_Part_Number (none) -> TLHY4400-AS12Z; Mouser Part Number 78-TLHR4400-AS12Z -> 78-TLHY4400-AS12Z; Mouser Price/Stock (none) -> https://pt.mouser.com/en/ProductDetail/Vishay-Semiconductor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; Supplier Link https://www.mouser.co.uk/ProductDetail/Vishay-Semiconductor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 -> https://pt.mouser.com/en/ProductDetail/Vishay-Semiconductor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
- LS1: Manufacturer Murata Electronics -> (none); Manufacturer Part Number PKMCS1818E20A0-R1 -> (none); Manufacturer_Name (none) -> Murata Electronics; Manufacturer_Part_Number (none) -> PKMCS1818E20A0-R1; Mouser Price/Stock (none) -> https://pt.mouser.com/en/ProductDetail/Murata-Electronics/P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; Supplier Link https://www.mouser.co.uk/ProductDetail/Murata-Electronics/P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 -> (none)
- R10, R9: Manufacturer Panasonic -> (none); Manufacturer Part Number ERJ-S03J470V -> (none); Manufacturer_Name (none) -> Vishay; Manufacturer_Part_Number (none) -> MCS04020C4709FE000; Mouser Part Number 667-ERJ-S03J470V -> 594-MCS04020C4709FE0; Mouser Price/Stock (none) -> https://pt.mouser.com/en/ProductDetail/Vishay-Beyschlag/MCS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; Supplier Link https://pt.mouser.com/ProductDetail/Panasonic/ERJ-S03J470V?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 -> https://pt.mouser.com/en/ProductDetail/Vishay-Beyschlag/MCS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
- R11: Manufacturer Vishay -> (none); Manufacturer Part Number RCA060310K0JNEA -> (none); Manufacturer_Name (none) -> Vishay; Manufacturer_Part_Number (none) -> MCS04020C1002FE000; Mouser Part Number 71-RCA060310K0JNEA -> 594-MCS04020C1002FE0; Mouser Price/Stock (none) -> https://pt.mouser.com/en/ProductDetail/Vishay-Beyschlag/MCS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; Supplier Link https://pt.mouser.com/ProductDetail/Vishay-Draloric/RCA0603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 -> https://pt.mouser.com/en/ProductDetail/Vishay-Beyschlag/MCS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
- R12: Manufacturer Vishay -> (none); Manufacturer_Name (none) -> Vishay; Manufacturer_Part_Number (none) -> MCS04020C1002FE000; Mouser Part Number 71-RCA060310K0JNEA -> 594-MCS04020C1002FE0; Mouser Price/Stock (none) -> https://pt.mouser.com/en/ProductDetail/Vishay-Beyschlag/MCS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; Supplier Link https://pt.mouser.com/ProductDetail/Vishay-Draloric/RCA0603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 -> https://pt.mouser.com/en/ProductDetail/Vishay-Beyschlag/MCS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
- R18, R19: Manufacturer Yageo -> (none); Manufacturer Part Number SR0603JR-7T33RL -> (none); Manufacturer_Name (none) -> Vishay; Manufacturer_Part_Number (none) -> MCS04020C1000FE000; Mouser Part Number 603-SR0603JR-7T33RL -> 594-MCS04020C1000FE0; Mouser Price/Stock (none) -> https://pt.mouser.com/en/ProductDetail/Vishay-Beyschlag/MCS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; Supplier Link https://pt.mouser.com/ProductDetail/YAGEO/SR0603JR-7T33RL?q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 -> https://pt.mouser.com/en/ProductDetail/Vishay-Beyschlag/MCS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
- R20: Manufacturer Yageo -> (none); Manufacturer Part Number AR0603FR-071ML -> (none); Manufacturer_Name (none) -> Vishay; Manufacturer_Part_Number (none) -> MCS04020C1002FE000; Mouser Part Number 603-AR0603FR-071ML -> 594-MCS04020C1002FE0; Mouser Price/Stock (none) -> https://pt.mouser.com/en/ProductDetail/Vishay-Beyschlag/MCS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; Supplier Link https://pt.mouser.com/ProductDetail/YAGEO/AR0603FR-071ML?qs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 -> https://pt.mouser.com/en/ProductDetail/Vishay-Beyschlag/MCS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
- R8: Manufacturer Vishay -> (none); Manufacturer Part Number CRCW0603100RJNEBC -> (none); Manufacturer_Name (none) -> Vishay; Manufacturer_Part_Number (none) -> MCS04020C1000FE000; Mouser Part Number 71-CRCW0603100RJNEBC -> 594-MCS04020C1000FE0; Mouser Price/Stock (none) -> https://pt.mouser.com/en/ProductDetail/Vishay-Beyschlag/MCS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; Supplier Link https://pt.mouser.com/ProductDetail/Vishay/CRCW0603100RJNEB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 -> https://pt.mouser.com/en/ProductDetail/Vishay-Beyschlag/MCS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
- U1: Manufacturer_Name (none) -> Mean Well; Manufacturer_Part_Number (none) -> IRM-01-3.3; Mouser Part Number (none) -> 709-IRM01-3.3; Mouser Price/Stock (none) -> https://pt.mouser.com/en/ProductDetail/MEAN-WELL/IRM-01-3.3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
Other:
- note removed: "Check the MCU pins again, for pull-ups, etc."
