File: hardware/gateway/rev2/gateway_rev2.kicad_pcb (KiCad board)
At the start: 2 copper layers, 94 x 78 mm, 68 parts, among them IC1 STM8L151K4T6, IC2 CC1101RGPR, IC5 MB85RC64TAPNF-G-BDERE1, J1 22-28-4044, J2 M20-9770342, U1 IRM-01-3.3, Y1 NX3225GA-26MHZ-TI

Commit message: EG-59 CRC Cheks and outputs generated.
Other:
- board text removed: "Check LEDs correct height in 3D model. Put the 230 V AC away from the low voltage paths, including GND plane."
